Commit message: Added the Kinect Sensor. Created a new robot with the Kinect attached to the head. Created a new launch file for the Kinect robot.

File: aurobot_description/urdf/common.xacro (robot description, xacro)
@@ -5,7 +5,7 @@
   <!-- ********** Right Arm ********** -->
   <!-- Gear Ratio Corrections: Divide transmission reductions by these factors (Nominally 1)-->
-  <property name="cal_r_shoulder_roll_gearing"   value="1.0"/>
-  <property name="cal_r_shoulder_lift_gearing"  value="1.0"/>
-  <property name="cal_r_upper_arm_roll_gearing" value="1.0"/>
+  <property name="cal_l_shoulder_roll_gearing"   value="1.0"/>
+  <property name="cal_l_shoulder_lift_gearing"  value="1.0"/>
+  <property name="cal_l_upper_arm_roll_gearing" value="1.0"/>
   <!-- Flag offsets: Add to the optical flag locations (Nominally 0) -->
   <property name="cal_r_shoulder_roll_flag"   value="0.0"/>

File: aurobot_description/urdf/shoulder/shoulder.transmission.xacro (robot description, xacro)
@@ -13,5 +13,5 @@
       <actuator name="${side}_shoulder_roll_motor">
         <hardwareInterface>hardware_interface/EffortJointInterface</hardwareInterface>
-        <mechanicalReduction>${13/3 * 250.532/17.19 / cal_r_shoulder_roll_gearing}</mechanicalReduction>
+        <mechanicalReduction>${13/3 * 250.532/17.19 / cal_l_shoulder_roll_gearing}</mechanicalReduction>
         <compensator k_belt="4000.0" mass_motor="0.05" kd_motor="15.0" lambda_motor="40.0" lambda_joint="40.0"
           lambda_combined="0.0"/>
@@ -26,5 +26,5 @@
       <actuator name="${side}_shoulder_lift_motor">
         <hardwareInterface>hardware_interface/EffortJointInterface</hardwareInterface>
-        <mechanicalReduction>${13/3 * 245.532/17.19 / cal_r_shoulder_lift_gearing}</mechanicalReduction>
+        <mechanicalReduction>${13/3 * 245.532/17.19 / cal_l_shoulder_lift_gearing}</mechanicalReduction>
         <compensator k_belt="4000.0" mass_motor="0.05" kd_motor="10.0" lambda_motor="60.0" lambda_joint="60.0"
           lambda_combined="0.0"/>
@@ -39,5 +39,5 @@
       <actuator name="${side}_upper_arm_roll_motor">
         <hardwareInterface>hardware_interface/EffortJointInterface</hardwareInterface>
-        <mechanicalReduction>${13/3 * 129.53/17.19 / cal_r_upper_arm_roll_gearing}</mechanicalReduction>
+        <mechanicalReduction>${13/3 * 129.53/17.19 / cal_l_upper_arm_roll_gearing}</mechanicalReduction>
       </actuator>
     </transmission>

File: aurobot_description/urdf/trunk/trunk.gazebo.xacro (robot description, xacro)
@@ -9,5 +9,9 @@
       <turnGravityOff>true</turnGravityOff>
     </gazebo>
-    <gazebo reference="trunk_joint">
+    <gazebo reference="trunk_left_joint">
+      <stopKd value="1.0"/>
+      <stopKp value="1000000.0"/>
+    </gazebo>
+    <gazebo reference="trunk_head_joint">
       <stopKd value="1.0"/>
       <stopKp value="1000000.0"/>

File: aurobot_description/urdf/trunk/trunk.urdf.xacro (robot description, xacro)
@@ -10,5 +10,5 @@
   <xacro:include filename="$(find aurobot_description)/urdf/common.xacro"/>
  <!-- ============================   Profiles   ============================ -->
-  <xacro:macro name="trunk" params="child">
+  <xacro:macro name="trunk" params="left_child head_child">
     <!-- Trunk link -->
     <link name="trunk_link">
@@ -32,6 +32,12 @@
     <joint name="trunk_left_joint" type="fixed">
       <parent link="trunk_link"/>
-      <child link="${child}"/>
+      <child link="${left_child}"/>
       <origin xyz="0 0.13790 1.22809" rpy="0 1.0471975512 1.5707963268"/>
+    </joint>
+    <joint name="trunk_head_joint" type="fixed">
+      <parent link="trunk_link"/>
+      <child link="${head_child}"/>
+      <!-- BRAYAN (16-05-2017): Temporalmente puesto como una cabeza adelantada. -->
+      <origin xyz="0.150 0 1.47" rpy="0 0 0"/>
     </joint>
     <!-- extensions   -->
