Commit message: PA10 joints' prefix changed from 'r_' to 'l_'. Fixed the error on controller loading.

File: aurobot_description/robots/aurobot.urdf.xacro (robot description, xacro)
@@ -31,11 +31,11 @@
   <xacro:base child="bearing_under_link"/>
   <xacro:bearing child="trunk_link"/>
-  <xacro:trunk child="r_shoulder_roll_link"/>
-  <!-- Add the right PA10 -->
-  <xacro:pa10_shoulder side="r" child="r_elbow_flex_link"/>
-  <xacro:pa10_upper_arm side="r" child="r_wrist_flex_link"/>
-  <xacro:pa10_forearm side="r" child="r_jr3_link"/>
+  <xacro:trunk child="l_shoulder_roll_link"/>
+  <!-- Add the left PA10 -->
+  <xacro:pa10_shoulder side="l" child="l_elbow_flex_link"/>
+  <xacro:pa10_upper_arm side="l" child="l_wrist_flex_link"/>
+  <xacro:pa10_forearm side="l" child="l_jr3_link"/>
   <!-- JR3 -->
-  <link name="r_jr3_link">
+  <link name="l_jr3_link">
   <inertial>
     <origin xyz="0 0 0" rpy="0 0 0"/>

Commit message: Added a head to the aurobot (without Kinect) to the new Trunk joint.

File: aurobot_description/robots/aurobot.urdf.xacro (robot description, xacro)
@@ -31,5 +31,29 @@
   <xacro:base child="bearing_under_link"/>
   <xacro:bearing child="trunk_link"/>
-  <xacro:trunk child="l_shoulder_roll_link"/>
+  <xacro:trunk left_child="l_shoulder_roll_link" head_child="head_link"/>
+  <!-- Head -->
+  <link name="head_link">
+    <inertial>
+      <origin xyz="0 0 1" rpy="0 0 0"/>
+      <mass value="1"/>
+      <inertia
+        ixx="1.0" ixy="0.0" ixz="0.0"
+        iyy="1.0" iyz="0.0"
+        izz="1.0"/>
+    </inertial>
+    <visual>
+      <origin xyz="-0.15 0 0.16" rpy="0 0 0"/>
+      <geometry>
+        <box size="0.3 0.3 0.3"/>
+      </geometry>
+      <material name="black"/>
+    </visual>
+    <collision>
+      <origin xyz="-0.15 0 0.16" rpy="0 0 0"/>
+      <geometry>
+        <box size="0.3 0.3 0.3"/>
+      </geometry>
+    </collision>
+  </link>
   <!-- Add the left PA10 -->
   <xacro:pa10_shoulder side="l" child="l_elbow_flex_link"/>

Commit message: Changed the orientation of the aurobot head_link to fit the camera view. Added a new package called "aurobot_utils". It holds now the script for transforming the camera point cloud topic to the world frame.

File: aurobot_description/robots/aurobot.urdf.xacro (robot description, xacro)
@@ -43,14 +43,14 @@
     </inertial>
     <visual>
-      <origin xyz="-0.15 0 0.16" rpy="0 0 0"/>
+      <origin xyz="0 0 0" rpy="0 0 0"/>
       <geometry>
-        <box size="0.3 0.3 0.3"/>
+        <box size="0.05 0.05 0.05"/>
       </geometry>
       <material name="black"/>
     </visual>
     <collision>
-      <origin xyz="-0.15 0 0.16" rpy="0 0 0"/>
+      <origin xyz="0 0 0" rpy="0 0 0"/>
       <geometry>
-        <box size="0.3 0.3 0.3"/>
+        <box size="0.05 0.05 0.05"/>
       </geometry>
     </collision>

File: aurobot_description/urdf/trunk/trunk.urdf.xacro (robot description, xacro)
@@ -38,6 +38,7 @@
       <parent link="trunk_link"/>
       <child link="${head_child}"/>
-      <!-- BRAYAN (16-05-2017): Temporalmente puesto como una cabeza adelantada. -->
-      <origin xyz="0.150 0 1.47" rpy="0 0 0"/>
+      <!-- BRAYAN (16-05-2017): Temporalmente puesto como una cabeza adelantada orientada hacia adelante.
+      -1.570796327 0 -1.570796327-->
+      <origin xyz="0.150 0 1.47" rpy="-2.042035225 0 -1.570796327"/>
     </joint>
     <!-- extensions   -->

Commit message: Added the Allegro left hand to the PA10. Updated the MoveIt demo.

File: aurobot_description/robots/aurobot.urdf.xacro (robot description, xacro)
@@ -21,4 +21,6 @@
   <xacro:include filename="$(find aurobot_description)/urdf/forearm/forearm.urdf.xacro"/>
   <xacro:include filename="$(find aurobot_description)/urdf/profiles/profiles.urdf.xacro"/>
+  <!-- Allegro left hand -->
+  <xacro:include filename="$(find aurobot_description)/urdf/hand/allegro/allegro_left.urdf.xacro"/>
   <!-- Joint the robot to the world -->
   <link name="world"/>
@@ -79,3 +81,10 @@
     </collision>
   </link>
+  <joint name="l_jr3_joint" type="fixed">
+    <parent link="l_jr3_link"/>
+    <child link="l_allegro_base_link"/>
+    <origin xyz="0 0 0.1" rpy="0 0 0"/>
+  </joint>
+  <!-- Allegro left hand -->
+  <xacro:allegro_left_hand/>
 </robot>

Commit message: Updated the robot colours. The Allegro left hand is now correctly oriented. Created new move group and end effector for the right pa10.

File: aurobot_description/robots/aurobot.urdf.xacro (robot description, xacro)
@@ -16,5 +16,9 @@
   <xacro:include filename="$(find aurobot_description)/urdf/robot-base/bearing/bearing.urdf.xacro"/>
   <xacro:include filename="$(find aurobot_description)/urdf/robot-base/trunk/trunk.urdf.xacro"/>
-  <!-- PA10 Arm -->
+  <!-- PA10 blue right arm -->
+  <xacro:include filename="$(find aurobot_description)/urdf/pa10-blue/shoulder/shoulder.urdf.xacro"/>
+  <xacro:include filename="$(find aurobot_description)/urdf/pa10-blue/upper_arm/upper_arm.urdf.xacro"/>
+  <xacro:include filename="$(find aurobot_description)/urdf/pa10-blue/forearm/forearm.urdf.xacro"/>
+  <!-- PA10 green left arm -->
   <xacro:include filename="$(find aurobot_description)/urdf/pa10-green/shoulder/shoulder.urdf.xacro"/>
   <xacro:include filename="$(find aurobot_description)/urdf/pa10-green/upper_arm/upper_arm.urdf.xacro"/>
@@ -32,5 +36,6 @@
   <xacro:base child="bearing_under_link"/>
   <xacro:bearing child="trunk_link"/>
-  <xacro:trunk left_child="pa10_green_shoulder_roll_link" head_child="head_link"/>
+  <xacro:trunk left_child="pa10_green_shoulder_roll_link"
+    head_child="head_link" right_child="pa10_blue_shoulder_roll_link"/>
   <!-- Head -->
   <link name="head_link">
@@ -57,9 +62,32 @@
     </collision>
   </link>
+  <!-- Add the right PA10 -->
+  <xacro:pa10_blue_shoulder child="pa10_blue_elbow_flex_link"/>
+  <xacro:pa10_blue_upper_arm child="pa10_blue_wrist_flex_link"/>
+  <xacro:pa10_blue_forearm child="r_jr3_link"/>
+  <!-- JR3 right -->
+  <link name="r_jr3_link">
+  <inertial>
+    <origin xyz="0 0 0" rpy="0 0 0"/>
+    <mass value="0.40"/>
+    <inertia ixx="0.012500"  ixy="0.000005"  ixz="0.000005" iyy="0.011431" iyz="0.000005" izz="0.012500"/>
+  </inertial>
+  <visual>
+    <geometry>
+    <mesh filename="package://aurobot_description/meshes/jr3/jr3.stl"/>
+    </geometry>
+    <material name="black"/>
+  </visual>
+  <collision>
+      <geometry>
+        <mesh filename="package://aurobot_description/meshes/jr3/jr3.stl"/>
+      </geometry>
+    </collision>
+  </link>
   <!-- Add the left PA10 -->
   <xacro:pa10_green_shoulder child="pa10_green_elbow_flex_link"/>
   <xacro:pa10_green_upper_arm child="pa10_green_wrist_flex_link"/>
   <xacro:pa10_green_forearm child="l_jr3_link"/>
-  <!-- JR3 -->
+  <!-- JR3 left -->
   <link name="l_jr3_link">
   <inertial>
@@ -76,5 +104,5 @@
   <collision>
       <geometry>
-    <mesh filename="package://aurobot_description/meshes/jr3/jr3.stl"/>
+        <mesh filename="package://aurobot_description/meshes/jr3/jr3.stl"/>
       </geometry>
     </collision>
@@ -83,5 +111,5 @@
     <parent link="l_jr3_link"/>
     <child link="l_allegro_base_link"/>
-    <origin xyz="0 0 0.1" rpy="0 0 0"/>
+    <origin xyz="0 0 0.1" rpy="0 0 3.1415926536"/>
   </joint>
   <!-- Allegro left hand -->

File: aurobot_description/urdf/pa10-blue/forearm/forearm.gazebo.xacro (robot description, xacro)
@@ -4,5 +4,5 @@
        xmlns:interface="http://playerstage.sourceforge.net/gazebo/xmlschema/#interface"
        xmlns:xacro="http://ros.org/wiki/xacro">
-  <xacro:macro name="pa10_forearm_gazebo">
+  <xacro:macro name="pa10_blue_forearm_gazebo">
     <!-- Wrist flex -->
     <gazebo reference="pa10_blue_wrist_flex_link">
@@ -10,5 +10,4 @@
       <mu1>0.2</mu1>
       <mu2>0.2</mu2>
-      <material>Gazebo/Green</material>
     </gazebo>
     <gazebo reference="pa10_blue_wrist_flex_joint">
@@ -21,5 +20,4 @@
       <mu1>0.2</mu1>
       <mu2>0.2</mu2>
-      <material>Gazebo/Grey</material>
     </gazebo>
     <gazebo reference="pa10_blue_wrist_roll_joint">

File: aurobot_description/urdf/pa10-blue/forearm/forearm.transmission.xacro (robot description, xacro)
@@ -5,5 +5,5 @@
        xmlns:xacro="http://ros.org/wiki/xacro">
   <!-- ============================   Forearm   ============================ -->
-  <xacro:macro name="pa10_forearm_transmission">
+  <xacro:macro name="pa10_blue_forearm_transmission">
     <!-- W1: Wrist flex , W2: Wrist roll -->
     <transmission name="pa10_blue_wrist_trans">

File: aurobot_description/urdf/pa10-blue/forearm/forearm.urdf.xacro (robot description, xacro)
@@ -24,7 +24,5 @@
           <mesh filename="package://aurobot_description/meshes/pa10-blue/forearm/W1.stl"/>
         </geometry>
-        <material name="">
-          <color rgba="0.33 0.96 0.53 1.5"/>
-        </material>
+        <material name="white"/>
       </visual>
       <collision>
@@ -40,5 +38,5 @@
       <origin xyz="0 0 0.195" rpy="0 0 0"/>
       <axis xyz="0 1 0"/>
-      <limit effort="0" lower="-2.878" upper="2.878" velocity="1.0"/>
+      <limit effort="1000.0" lower="-2.878" upper="2.878" velocity="0.628"/>
     </joint>
     <!-- W2: Wrist roll -->
@@ -54,7 +52,5 @@
           <mesh filename="package://aurobot_description/meshes/pa10-blue/forearm/W2.stl"/>
         </geometry>
-        <material name="">
-          <color rgba="0.34 0.35 0.36 1.0"/>
-        </material>
+        <material name="blue"/>
       </visual>
       <collision>
@@ -68,7 +64,7 @@
       <parent link="pa10_blue_wrist_roll_link"/>
       <child link="${child}"/>
-      <origin xyz="0 0 0" rpy="0 0 0"/>
+      <origin xyz="0 0 0.075" rpy="0 0 0"/>
       <axis xyz="0 0 1"/>
-      <limit effort="0" lower="-2.878" upper="2.878" velocity="1.0"/>
+      <limit effort="1000.0" lower="-2.878" upper="2.878" velocity="0.628"/>
     </joint>
     <!-- extensions-->

File: aurobot_description/urdf/pa10-blue/shoulder/shoulder.gazebo.xacro (robot description, xacro)
@@ -10,5 +10,4 @@
       <mu1>0.2</mu1>
       <mu2>0.2</mu2>
-      <material>Gazebo/Grey</material>
     </gazebo>
     <gazebo reference="pa10_blue_shoulder_roll_joint">
@@ -19,5 +18,4 @@
     <gazebo reference="pa10_blue_shoulder_lift_link">
       <turnGravityOff>true</turnGravityOff>
-      <material>Gazebo/Green</material>
     </gazebo>
     <gazebo reference="pa10_blue_shoulder_lift_joint">
@@ -30,5 +28,4 @@
       <mu1>0.2</mu1>
       <mu2>0.2</mu2>
-      <material>Gazebo/Grey</material>
     </gazebo>
     <gazebo reference="pa10_blue_upper_arm_roll_joint">

File: aurobot_description/urdf/pa10-blue/shoulder/shoulder.urdf.xacro (robot description, xacro)
@@ -24,7 +24,5 @@
             <mesh filename="package://aurobot_description/meshes/pa10-blue/shoulder/S1.stl"/>
         </geometry>
-        <material name="">
-          <color rgba="0.34 0.35 0.36 1.0"/>
-        </material>
+        <material name="blue"/>
       </visual>
       <collision>
@@ -40,5 +38,7 @@
       <origin xyz="0 0 0.2" rpy="0 0 0"/>
       <axis xyz="0 0 1"/>
-      <limit effort="0" lower="-3.089" upper="3.089" velocity="1.0"/>
+      <limit effort="1000.0" lower="-3.089" upper="3.089" velocity="0.1"/>
+      <cfm>0.7</cfm>
+      <damping>10.0</damping>
     </joint>
     <!-- S2: Shoulder lift -->
@@ -54,7 +54,5 @@
           <mesh filename="package://aurobot_description/meshes/pa10-blue/shoulder/S2.stl"/>
         </geometry>
-        <material name="">
-          <color rgba="0.33 0.96 0.53 1.5"/>
-        </material>
+        <material name="white"/>
       </visual>
       <collision>
@@ -70,5 +68,7 @@
       <origin xyz="0 0 0.117" rpy="0 0 0"/>
       <axis xyz="0 1 0"/>
-      <limit effort="0" lower="-1.64" upper="1.64" velocity="1.0"/>
+      <limit effort="1000.0" lower="-1.64" upper="1.64" velocity="0.1"/>
+      <cfm>0.7</cfm>
+      <damping>10.0</damping>
     </joint>
     <!-- S3: Upperarm roll -->
@@ -84,7 +84,5 @@
           <mesh filename="package://aurobot_description/meshes/pa10-blue/shoulder/S3.stl"/>
         </geometry>
-        <material name="">
-          <color rgba="0.34 0.35 0.36 1.0"/>
-        </material>
+        <material name="blue"/>
       </visual>
       <collision>
@@ -100,5 +98,7 @@
       <origin xyz="0 0 0.317" rpy="0 0 0"/>
       <axis xyz="0 0 1"/>
-      <limit effort="0" lower="-3.036" upper="3.036" velocity="1.0"/>
+      <limit effort="1000.0" lower="-3.036" upper="3.036" velocity="0.1"/>
+      <cfm>0.7</cfm>
+      <damping>10.0</damping>
     </joint>
     <!-- extensions -->

File: aurobot_description/urdf/pa10-blue/upper_arm/upper_arm.gazebo.xacro (robot description, xacro)
@@ -10,5 +10,4 @@
       <mu1>0.2</mu1>
       <mu2>0.2</mu2>
-      <material>Gazebo/Green</material>
     </gazebo>
     <gazebo reference="pa10_blue_elbow_flex_joint">
@@ -21,5 +20,4 @@
       <mu1>0.2</mu1>
       <mu2>0.2</mu2>
-      <material>Gazebo/Grey</material>
     </gazebo>
     <gazebo reference="pa10_blue_forearm_roll_joint">

File: aurobot_description/urdf/pa10-blue/upper_arm/upper_arm.transmission.xacro (robot description, xacro)
@@ -5,5 +5,5 @@
        xmlns:xacro="http://ros.org/wiki/xacro">
   <!-- ============================   Upper Arm   ============================ -->
-  <xacro:macro name="pa10_upper_arm_transmission">
+  <xacro:macro name="pa10_blue_upper_arm_transmission">
     <!-- E1: Elbow flex -->
     <transmission name="pa10_blue_elbow_flex_trans">

File: aurobot_description/urdf/pa10-blue/upper_arm/upper_arm.urdf.xacro (robot description, xacro)
@@ -24,7 +24,5 @@
           <mesh filename="package://aurobot_description/meshes/pa10-blue/upper_arm/E1.stl"/>
         </geometry>
-        <material name="">
-          <color rgba="0.33 0.96 0.53 1.5"/>
-        </material>
+        <material name="white"/>
       </visual>
       <collision>
@@ -40,5 +38,7 @@
       <origin xyz="0 0 0.133" rpy="0 0 0"/>
       <axis xyz="0 1 0"/>
-      <limit effort="0" lower="-2.39" upper="2.39" velocity="1.0"/>
+      <limit effort="1000.0" lower="-2.39" upper="2.39" velocity="0.2"/>
+      <cfm>0.7</cfm>
+      <damping>10.0</damping>
     </joint>
     <!-- E2: Forearm_roll -->
@@ -54,7 +54,5 @@
           <mesh filename="package://aurobot_description/meshes/pa10-blue/upper_arm/E2.stl"/>
         </geometry>
-        <material name="">
-          <color rgba="0.34 0.35 0.36 1.0"/>
-        </material>
+        <material name="blue"/>
       </visual>
       <collision>
@@ -70,5 +68,7 @@
       <origin xyz="0 0 0.285" rpy="0 0 0"/>
       <axis xyz="0 0 1"/>
-      <limit effort="0" lower="-4.45" upper="4.45" velocity="1.0"/>
+      <limit effort="1000.0" lower="-4.45" upper="4.45" velocity="0.2"/>
+      <cfm>0.7</cfm>
+      <damping>10.0</damping>
     </joint>
     <!-- extensions-->

File: aurobot_description/urdf/robot-base/base/base.urdf.xacro (robot description, xacro)
@@ -22,5 +22,5 @@
           <mesh filename="package://aurobot_description/meshes/robot-base/base/base_down.stl" scale="0.001 0.001 0.001"/>
         </geometry>
-        <material name="blue"/>
+        <material name="grey"/>
       </visual>
       <collision>
@@ -45,5 +45,5 @@
           <mesh filename="package://aurobot_description/meshes/robot-base/base/base_up.stl" scale="0.001 0.001 0.001"/>
         </geometry>
-        <material name="blue"/>
+        <material name="grey"/>
       </visual>
       <collision>

File: aurobot_description/urdf/robot-base/bearing/bearing.urdf.xacro (robot description, xacro)
@@ -22,5 +22,5 @@
           <mesh filename="package://aurobot_description/meshes/robot-base/bearing/bearing_under.stl" scale="0.001 0.001 0.001"/>
         </geometry>
-        <material name="blue"/>
+        <material name="grey"/>
       </visual>
       <collision>
@@ -45,5 +45,5 @@
           <mesh filename="package://aurobot_description/meshes/robot-base/bearing/bearing.stl" scale="0.001 0.001 0.001"/>
         </geometry>
-        <material name="blue"/>
+        <material name="green"/>
       </visual>
       <collision>
@@ -68,5 +68,5 @@
           <mesh filename="package://aurobot_description/meshes/robot-base/bearing/bearing_above.stl" scale="0.001 0.001 0.001"/>
         </geometry>
-        <material name="blue"/>
+        <material name="grey"/>
       </visual>
       <collision>

File: aurobot_description/urdf/robot-base/profiles/profiles.urdf.xacro (robot description, xacro)
@@ -22,5 +22,5 @@
           <mesh filename="package://aurobot_description/meshes/robot-base/profiles/profiles.stl" scale="0.001 0.001 0.001"/>
         </geometry>
-        <material name="blue"/>
+        <material name="grey"/>
       </visual>
       <collision>

File: aurobot_description/urdf/robot-base/trunk/trunk.urdf.xacro (robot description, xacro)
@@ -10,5 +10,5 @@
   <xacro:include filename="$(find aurobot_description)/urdf/common.xacro"/>
  <!-- ============================   Profiles   ============================ -->
-  <xacro:macro name="trunk" params="left_child head_child">
+  <xacro:macro name="trunk" params="left_child head_child right_child">
     <!-- Trunk link -->
     <link name="trunk_link">
@@ -22,5 +22,5 @@
           <mesh filename="package://aurobot_description/meshes/robot-base/trunk/trunk.stl" scale="0.001 0.001 0.001"/>
         </geometry>
-        <material name="blue"/>
+        <material name="grey"/>
       </visual>
       <collision>
@@ -42,4 +42,9 @@
       <origin xyz="0.150 0 1.47" rpy="-2.042035225 0 -1.570796327"/>
     </joint>
+    <joint name="trunk_right_joint" type="fixed">
+      <parent link="trunk_link"/>
+      <child link="${right_child}"/>
+      <origin xyz="0 -0.13790 1.22809" rpy="0 -1.0471975512 1.5707963268"/>
+    </joint>
     <!-- extensions   -->
     <xacro:trunk_gazebo/>
