Commit message: Some fixes to aurobot_plan. Redefinition of the allegro to run the shadow robot.

File: aurobot_description/robots/aurobot_shadow.urdf.xacro (robot description, xacro)
@@ -27,5 +27,5 @@
   <xacro:include filename="$(find aurobot_description)/urdf/hand/allegro/allegro_left.urdf.xacro"/>
   <!-- Shadow right hand arm -->
-  <!-- sr_destriptor repository is in https://github.com/shadow-robot/sr-ros-interface.git -->
+  <!-- sr_description is in https://github.com/shadow-robot/sr_common/tree/kinetic-devel -->
   <xacro:include filename="$(find sr_description)/materials.urdf.xacro" />
   <xacro:include filename="$(find sr_description)/hand/xacro/full_hand.urdf.xacro" />

File: aurobot_description/urdf/hand/allegro/allegro_left.urdf.xacro (robot description, xacro)
@@ -200,4 +200,5 @@
   <!-- ============================================================================= -->
   <xacro:macro name="allegro_finger" params="finger_num offset_origin_x offset_origin_y offset_origin_z finger_angle_r">
+  <!-- <xacro:macro name="finger" params="finger_num offset_origin_x offset_origin_y offset_origin_z finger_angle_r"> -->
     <!-- [LINK 0, 4, 8] -->
     <link name="l_allegro_link_${finger_num*4+0}">
@@ -373,4 +374,5 @@
     />
     <!-- FINGERS -->
+    <!-- <xacro:finger  -->
     <xacro:allegro_finger
       finger_num=     "2"
@@ -380,4 +382,5 @@
       finger_angle_r=   "-${5.0*DEG2RAD}"
     />
+    <!-- <xacro:finger  -->
     <xacro:allegro_finger
       finger_num=     "1"
@@ -387,4 +390,5 @@
       finger_angle_r=   "0.0"
     />
+    <!-- <xacro:finger  -->
     <xacro:allegro_finger
       finger_num=     "0"

Commit message: New gazebo file with the whole aurobot configuration. Changed some robot parameters to be equal to the green PA10 manual. The move left pa10 script now activates the brakes after holding a new position. Since the thumb is having an unexpcted behaviour, the pre grasp position is in is upper limit.

File: aurobot_description/robots/aurobot_shadow.urdf.xacro (robot description, xacro)
@@ -74,16 +74,16 @@
   <!-- JR3 left -->
   <link name="l_jr3_link">
-  <inertial>
-    <origin xyz="0 0 0" rpy="0 0 0"/>
-    <mass value="0.40"/>
-    <inertia ixx="0.012500"  ixy="0.000005"  ixz="0.000005" iyy="0.011431" iyz="0.000005" izz="0.012500"/>
-  </inertial>
-  <visual>
-    <geometry>
-    <mesh filename="package://aurobot_description/meshes/jr3/jr3.stl"/>
-    </geometry>
-    <material name="black"/>
-  </visual>
-  <collision>
+    <inertial>
+      <origin xyz="0 0 0" rpy="0 0 0"/>
+      <mass value="0.40"/>
+      <inertia ixx="0.012500"  ixy="0.000005"  ixz="0.000005" iyy="0.011431" iyz="0.000005" izz="0.012500"/>
+    </inertial>
+    <visual>
+      <geometry>
+      <mesh filename="package://aurobot_description/meshes/jr3/jr3.stl"/>
+      </geometry>
+      <material name="black"/>
+    </visual>
+    <collision>
       <geometry>
         <mesh filename="package://aurobot_description/meshes/jr3/jr3.stl"/>
@@ -94,5 +94,7 @@
     <parent link="l_jr3_link"/>
     <child link="l_allegro_base_link"/>
-    <origin xyz="0 0 0.1" rpy="0 0 3.1415926536"/>
+      <!-- BRAYAN (12/07/2017): Medimos y no tiene 10cm, son 4.7cm goma + jr3 + placa
+       <origin xyz="0 0 0.1" rpy="0 0 3.1415926536"/> -->
+    <origin xyz="0 0 0.047" rpy="0 0 3.1415926536"/>
   </joint>
   <!-- Allegro left hand -->
@@ -104,16 +106,16 @@
   <!-- JR3 right -->
   <link name="r_jr3_link">
-  <inertial>
-    <origin xyz="0 0 0" rpy="0 0 0"/>
-    <mass value="0.40"/>
-    <inertia ixx="0.012500"  ixy="0.000005"  ixz="0.000005" iyy="0.011431" iyz="0.000005" izz="0.012500"/>
-  </inertial>
-  <visual>
-    <geometry>
-    <mesh filename="package://aurobot_description/meshes/jr3/jr3.stl"/>
-    </geometry>
-    <material name="black"/>
-  </visual>
-  <collision>
+    <inertial>
+      <origin xyz="0 0 0" rpy="0 0 0"/>
+      <mass value="0.40"/>
+      <inertia ixx="0.012500"  ixy="0.000005"  ixz="0.000005" iyy="0.011431" iyz="0.000005" izz="0.012500"/>
+    </inertial>
+    <visual>
+      <geometry>
+      <mesh filename="package://aurobot_description/meshes/jr3/jr3.stl"/>
+      </geometry>
+      <material name="black"/>
+    </visual>
+    <collision>
       <geometry>
         <mesh filename="package://aurobot_description/meshes/jr3/jr3.stl"/>

File: aurobot_description/urdf/hand/allegro/allegro_left.urdf.xacro (robot description, xacro)
@@ -40,6 +40,6 @@
   <xacro:property name="limit_3_up" value="1.718" />
   <xacro:property name="limit_3_low" value=" -0.327" />
-  <xacro:property name="limit_0_t_up" value="1.496" />
-  <xacro:property name="limit_0_t_low" value="0.363" />
+  <xacro:property name="limit_0_t_up" value="1.4968131524486665" />
+  <xacro:property name="limit_0_t_low" value="0.3635738998060688" />
   <xacro:property name="limit_1_t_up" value="1.263" />
   <xacro:property name="limit_1_t_low" value="-0.205" />
@@ -82,5 +82,6 @@
     <joint name="l_allegro_joint_${finger_num*4}" type="revolute">
       <axis xyz="+1 0 0"/>
-      <limit effort="15" velocity="7" lower="${limit_0_t_low-joint_safety_margin}" upper="${limit_0_t_up-joint_safety_margin}" />
+      <!-- <limit effort="15" velocity="7" lower="${limit_0_t_low-joint_safety_margin}" upper="${limit_0_t_up-joint_safety_margin}" /> -->
+      <limit effort="15" velocity="7" lower="${limit_0_t_low}" upper="${limit_0_t_up}" />
       <parent link="l_allegro_base_link"/>
       <child link="l_allegro_link_${finger_num*4+0}"/>

File: aurobot_description/urdf/pa10-green/forearm/forearm.urdf.xacro (robot description, xacro)
@@ -38,5 +38,5 @@
       <origin xyz="0 0 0.05" rpy="0 0 0"/>
       <axis xyz="0 1 0"/>
-      <limit effort="1000.0" lower="-2.88" upper="2.88" velocity="0.628"/>
+      <limit effort="1000.0" lower="-2.8797932658" upper="2.8797932658" velocity="0.628"/>
       <cfm>0.7</cfm>
     </joint>
@@ -65,7 +65,9 @@
       <parent link="pa10_green_wrist_roll_link"/>
       <child link="${child}"/>
-      <origin xyz="0 0 0.050" rpy="0 0 0"/>
+      <!-- BRAYAN (12/07/2017): Segun el manual nos falta 0.03 <origin xyz="0 0 0.050" rpy="0 0 0"/> -->
+      <origin xyz="0 0 0.080" rpy="0 0 0"/>
       <axis xyz="0 0 1"/>
-      <limit effort="1000.0" lower="-2.0" upper="2.28" velocity="0.628"/>
+      <!-- BRAYAN (13/07/2017): gran cambio en lower y upper, casi el doble hemos puesto -->
+      <limit effort="1000.0" lower="-6.2831853072" upper="6.2831853072" velocity="0.628"/>
       <cfm>0.7</cfm>
     </joint>

File: aurobot_description/urdf/pa10-green/shoulder/shoulder.urdf.xacro (robot description, xacro)
@@ -34,7 +34,8 @@
       <parent link="pa10_green_shoulder_roll_link"/>
       <child link="pa10_green_shoulder_lift_link"/>
-      <origin xyz="0 0 0.201" rpy="0 0 0"/>
+      <!-- BRAYAN (12/07/2017): Segun el manual nos sobra 0.001 <origin xyz="0 0 0.201" rpy="0 0 0"/> -->
+      <origin xyz="0 0 0.20" rpy="0 0 0"/>
       <axis xyz="0 0 1"/>
-      <limit effort="1000.0" lower="-3.09" upper="3.09" velocity="0.1"/>
+      <limit effort="1000.0" lower="-3.089232776" upper="3.089232776" velocity="0.1"/>
       <cfm>0.7</cfm>
       <damping>10.0</damping>
@@ -66,5 +67,5 @@
       <origin xyz="0 0 0.115" rpy="0 0 0"/>
       <axis xyz="0 1 0"/>
-      <limit effort="1000.0" lower="-1.59" upper="1.59" velocity="0.1"/>
+      <limit effort="1000.0" lower="-1.5882496193" upper="1.5882496193" velocity="0.1"/>
       <cfm>0.7</cfm>
       <damping>10.0</damping>
@@ -94,5 +95,5 @@
       <axis xyz="0 0 1"/>
       <origin xyz="0 0 0.325" rpy="0 0 0"/>
-      <limit effort="1000.0" lower="-3.04" upper="3.04" velocity="0.2"/>
+      <limit effort="1000.0" lower="-3.0368728985" upper="3.0368728985" velocity="0.2"/>
       <cfm>0.7</cfm>
       <damping>10.0</damping>

File: aurobot_description/urdf/pa10-green/upper_arm/upper_arm.urdf.xacro (robot description, xacro)
@@ -38,5 +38,5 @@
       <origin xyz="0 0 0.125" rpy="0 0 0"/>
       <axis xyz="0 1 0"/>
-      <limit effort="1000.0" lower="-2.39" upper="2.39" velocity="0.2"/>
+      <limit effort="1000.0" lower="-2.3911010752" upper="2.3911010752" velocity="0.2"/>
       <cfm>0.7</cfm>
       <damping>10.0</damping>
@@ -66,5 +66,6 @@
       <axis xyz="0 0 1"/>
       <origin xyz="0 0 0.450" rpy="0 0 0"/>
-      <limit effort="1000.0" lower="-2.0" upper="2.0" velocity="0.628"/>
+      <!-- BRAYAN (13/07/2017): gran cambio en lower y upper, casi el doble hemos puesto -->
+      <limit effort="1000.0" lower="-4.4505895926" upper="4.4505895926" velocity="0.628"/>
     </joint>
     <!-- extensions-->

File: aurobot_description/urdf/robot-base/trunk/trunk.urdf.xacro (robot description, xacro)
@@ -38,9 +38,9 @@
       <parent link="trunk_link"/>
       <child link="${head_child}"/>
-      <!-- BRAYAN (16-05-2017): Temporalmente puesto como una cabeza adelantada orientada hacia adelante.
-      -1.570796327 0 -1.570796327-->
+      <!-- BRAYAN (16-05-2017): Temporalmente puesto como una cabeza adelantada orientada hacia adelante -->
       <!-- <origin xyz="0.045 -0.025 1.71" rpy="-2.2689280276 0 -1.570796327"/> -->
-      <!-- BRAYAN (10/07/2017): posicion a la izquierda. Tiene rotado en Z unos 180 + 3 grados de desviacion -->
-      <origin xyz="0.717 1.5334 1.731" rpy="-1.9722220548 0 3.1590459461"/>
+      <!-- BRAYAN (10/07/2017): posicion a la izquierda. Tiene en Roll (X) 109 negativos.
+        Tiene rotado en Yaw (Z) unos 180 + 1 grados de desviacion -->
+      <origin xyz="0.71 1.526 1.793" rpy="-2.0071286398 0 3.1538099584"/>
     </joint>
     <joint name="trunk_right_joint" type="fixed">
