Commit message: Added new PA10 (Green) model. It's an old one but seems to be more visually similar to the real robot. Changed the PA10 (Green) model definition. Origins set to 0,0,0 except for joints, where the manual distances are used.

File: aurobot_description/robots/aurobot_shadow.urdf.xacro (robot description, xacro)
@@ -44,4 +44,56 @@
   <xacro:trunk left_child="pa10_green_shoulder_roll_link"
     head_child="head_link" right_child="pa10_blue_shoulder_roll_link"/>
+  <!-- Cono Pecho -->
+  <link name="cone_trunk_link">
+    <inertial>
+      <origin xyz="0.27501 0.0 1.328" rpy="0 ${pi/2} 0 "/>
+      <mass value="1"/>
+      <inertia
+        ixx="1.0" ixy="0.0" ixz="0.0"
+        iyy="1.0" iyz="0.0"
+        izz="1.0"/>
+    </inertial>
+    <visual>
+      <origin xyz="0.27501 0.0 1.328" rpy="0 ${pi/2} 0"/>
+      <geometry>
+        <cylinder radius="0.045" length="0.25"/>
+      </geometry>
+      <material name="Cyan">
+        <color rgba="0 1.0 1.0 0.5"/>
+      </material>
+    </visual>
+    <collision>
+      <origin xyz="0.27501 0.0 1.328" rpy="0 ${pi/2} 0"/>
+      <geometry>
+        <cylinder radius="0.045" length="0.25"/>
+      </geometry>
+    </collision>
+  </link>
+  <!-- Cono2 Pecho -->
+  <link name="cone2_trunk_link">
+    <inertial>
+      <origin xyz="0.550 0.105 1.3225" rpy="0 0 0 "/>
+      <mass value="1"/>
+      <inertia
+        ixx="1.0" ixy="0.0" ixz="0.0"
+        iyy="1.0" iyz="0.0"
+        izz="1.0"/>
+    </inertial>
+    <visual>
+      <origin xyz="0.550 0.105 1.3225" rpy="0 0 0"/>
+      <geometry>
+        <cylinder radius="0.045" length="0.25"/>
+      </geometry>
+      <material name="Cyan">
+        <color rgba="0 1.0 1.0 0.3"/>
+      </material>
+    </visual>
+    <collision>
+      <origin xyz="0.550 0.105 1.3225" rpy="0 0 0"/>
+      <geometry>
+        <cylinder radius="0.045" length="0.25"/>
+      </geometry>
+    </collision>
+  </link>
   <!-- Head -->
   <link name="head_link">
@@ -57,5 +109,5 @@
       <origin xyz="0 0 0" rpy="0 0 0"/>
       <geometry>
-        <box size="0.05 0.05 0.05"/>
+        <box size="0.025 0.025 0.025"/>
       </geometry>
       <material name="black"/>
@@ -64,5 +116,5 @@
       <origin xyz="0 0 0" rpy="0 0 0"/>
       <geometry>
-        <box size="0.05 0.05 0.05"/>
+        <box size="0.025 0.025 0.025"/>
       </geometry>
     </collision>
@@ -81,11 +133,12 @@
     <visual>
       <geometry>
-      <mesh filename="package://aurobot_description/meshes/jr3/jr3.stl"/>
+        <!-- BRAYAN (22/11/2017): Escalamos esta pieza que en el STL mide menos de la realidad -->
+        <mesh filename="package://aurobot_description/meshes/jr3/jr3.stl" scale="1 1 8"/>
       </geometry>
-      <material name="black"/>
+      <material name="grey"/>
     </visual>
     <collision>
       <geometry>
-        <mesh filename="package://aurobot_description/meshes/jr3/jr3.stl"/>
+        <mesh filename="package://aurobot_description/meshes/jr3/jr3.stl" scale="1 1 8"/>
       </geometry>
     </collision>
@@ -94,7 +147,9 @@
     <parent link="l_jr3_link"/>
     <child link="l_allegro_base_link"/>
-      <!-- BRAYAN (12/07/2017): Medimos y no tiene 10cm, son 4.7cm goma + jr3 + placa
+      <!-- BRAYAN (12/07/2017): Medimos y no tiene 10cm, son 4.7cm placa + jr3 + placa
        <origin xyz="0 0 0.1" rpy="0 0 3.1415926536"/> -->
-    <origin xyz="0 0 0.047" rpy="0 0 3.1415926536"/>
+      <!-- BRAYAN (22/11/2017): Realmente son 4cm, porque 0.7cm primeros son de PA10
+       <origin xyz="0 0 0.047" rpy="0 0 3.1415926536"/> -->
+    <origin xyz="0 0 0.04042" rpy="0 0 3.1415926536"/>
   </joint>
   <!-- Allegro left hand -->
@@ -115,5 +170,5 @@
       <mesh filename="package://aurobot_description/meshes/jr3/jr3.stl"/>
       </geometry>
-      <material name="black"/>
+      <material name="grey"/>
     </visual>
     <collision>

File: aurobot_description/urdf/hand/allegro/allegro_left.urdf.xacro (robot description, xacro)
@@ -370,5 +370,6 @@
     <!-- BASE -->
     <link name="l_allegro_base_link">
-      <inertial> <!-- BRAYAN (03/07/2017): Changed to be equal to those on the allegro ros package-->
+      <inertial> <!-- BRAYAN (03/07/2017): Changed to be equal to those on the allegro ros package -->
+          <!-- BRAYAN (22/11/2017): quitamos este desplazamiento del origin <origin xyz="0 0 ${base_link_z/2}" rpy="0 0 0"/>-->
           <origin xyz="0 0 ${base_link_z/2}" rpy="0 0 0"/>
           <mass value="0.4154"/>

File: aurobot_description/urdf/pa10-green/forearm/forearm.urdf.xacro (robot description, xacro)
@@ -11,23 +11,22 @@
   <xacro:include filename="$(find aurobot_description)/urdf/common.xacro"/>
   <!-- ============================   Forearm   ============================ -->
+  <!-- BRAYAN (22/11/2017): Dejamos origin a 0,0,0 en todo lo que no sea joint -->
   <xacro:macro name="pa10_green_forearm" params="child" >
     <!-- W1: Wrist flex -->
     <link name="pa10_green_wrist_flex_link">
       <inertial>
-        <origin xyz="0 -0.0432 0.03" rpy="0 0 0"/>
         <mass value="3.45"/>
+        <origin xyz="0 0 0" rpy="0 0 0"/>
         <inertia ixx="0.076687"  ixy="0.000005"  ixz="0.000960" iyy="0.077392" iyz="0.000005" izz="0.006233"/>
       </inertial>
       <visual>
-        <origin xyz="0 0 0.03" rpy="0 0 0"/>
         <geometry>
-          <mesh filename="package://aurobot_description/meshes/pa10-green/forearm/W1.dae"/>
+          <mesh filename="package://aurobot_description/meshes/pa10-green/forearm/pa10_05.stl"/>
         </geometry>
         <material name="green"/>
       </visual>
       <collision>
-        <origin xyz="0 0 0.03" rpy="0 0 0"/>
         <geometry>
-          <mesh filename="package://aurobot_description/meshes/pa10-green/forearm/W1.stl"/>
+          <mesh filename="package://aurobot_description/meshes/pa10-green/forearm/pa10_05.stl"/>
         </geometry>
       </collision>
@@ -36,5 +35,6 @@
       <parent link="pa10_green_wrist_flex_link"/>
       <child link="pa10_green_wrist_roll_link"/>
-      <origin xyz="0 0 0.05" rpy="0 0 0"/>
+      <!-- BRAYAN (22/11/2017): Recalculo mas preciso <origin xyz="0 0 0.05" rpy="0 0 0"/> -->
+      <origin xyz="0 0 0.23643" rpy="0 0 0"/>
       <axis xyz="0 1 0"/>
       <limit effort="1000.0" lower="-2.8797932658" upper="2.8797932658" velocity="0.628"/>
@@ -44,19 +44,17 @@
     <link name="pa10_green_wrist_roll_link">
       <inertial>
-        <origin xyz="0 0.003 -0.0175" rpy="0 0 0"/>
         <mass value="1.46"/>
+        <origin xyz="0 0 0" rpy="0 0 0"/>
         <inertia ixx="0.012500"  ixy="0.000005"  ixz="0.000005" iyy="0.011431" iyz="0.000005" izz="0.012500"/>
       </inertial>
       <visual>
-        <origin xyz="0 0.0 -0.0175" rpy="0 0 0"/>
         <geometry>
-          <mesh filename="package://aurobot_description/meshes/pa10-green/forearm/W2.dae"/>
+          <mesh filename="package://aurobot_description/meshes/pa10-green/forearm/pa10_06.stl"/>
         </geometry>
         <material name="blue"/>
       </visual>
       <collision>
-        <origin xyz="0 0.0 -0.0175" rpy="0 0 0"/>
         <geometry>
-          <mesh filename="package://aurobot_description/meshes/pa10-green/forearm/W2.stl"/>
+          <mesh filename="package://aurobot_description/meshes/pa10-green/forearm/pa10_06.stl"/>
         </geometry>
       </collision>

File: aurobot_description/urdf/pa10-green/shoulder/shoulder.urdf.xacro (robot description, xacro)
@@ -11,4 +11,5 @@
   <xacro:include filename="$(find aurobot_description)/urdf/common.xacro"/>
  <!-- ============================   Shoulder   ============================ -->
+  <!-- BRAYAN (22/11/2017): Dejamos origin a 0,0,0 en todo lo que no sea joint -->
   <xacro:macro name="pa10_green_shoulder" params="child">
     <!-- S1: Shoulder roll -->
@@ -21,5 +22,5 @@
       <visual>
         <geometry>
-          <mesh filename="package://aurobot_description/meshes/pa10-green/shoulder/S1.dae"/>
+          <mesh filename="package://aurobot_description/meshes/pa10-green/shoulder/pa10_00.stl"/>
         </geometry>
         <material name="blue"/>
@@ -27,5 +28,5 @@
       <collision>
         <geometry>
-          <mesh filename="package://aurobot_description/meshes/pa10-green/shoulder/S1.stl"/>
+          <mesh filename="package://aurobot_description/meshes/pa10-green/shoulder/pa10_00.stl"/>
         </geometry>
       </collision>
@@ -34,6 +35,6 @@
       <parent link="pa10_green_shoulder_roll_link"/>
       <child link="pa10_green_shoulder_lift_link"/>
-      <!-- BRAYAN (12/07/2017): Segun el manual nos sobra 0.001 <origin xyz="0 0 0.201" rpy="0 0 0"/> -->
-      <origin xyz="0 0 0.20" rpy="0 0 0"/>
+      <!-- BRAYAN (22/11/2017): Recalculo mas preciso <origin xyz="0 0 0.20" rpy="0 0 0"/> -->
+      <origin xyz="0 0 0.20137" rpy="0 0 0"/>
       <axis xyz="0 0 1"/>
       <limit effort="1000.0" lower="-3.089232776" upper="3.089232776" velocity="0.1"/>
@@ -45,18 +46,16 @@
       <inertial>
         <mass value="9.78"/>
-        <origin xyz="0 0 0.115" rpy="0 0 0"/>
+        <origin xyz="0 0 0" rpy="0 0 0"/>
         <inertia ixx="0.110697"  ixy="0.000005"  ixz="0.000345" iyy="0.084268" iyz="0.000518" izz="0.054080"/>
       </inertial>
       <visual>
-        <origin xyz="0 0 0.115" rpy="0 0 0"/>
         <geometry>
-          <mesh filename="package://aurobot_description/meshes/pa10-green/shoulder/S2.dae"/>
+          <mesh filename="package://aurobot_description/meshes/pa10-green/shoulder/pa10_01.stl"/>
         </geometry>
         <material name="green"/>
       </visual>
       <collision>
-        <origin xyz="0 0 0.115" rpy="0 0 0"/>
         <geometry>
-          <mesh filename="package://aurobot_description/meshes/pa10-green/shoulder/S2.stl" />
+          <mesh filename="package://aurobot_description/meshes/pa10-green/shoulder/pa10_01.stl"/>
         </geometry>
       </collision>
@@ -65,5 +64,6 @@
       <parent link="pa10_green_shoulder_lift_link"/>
       <child link="pa10_green_upper_arm_roll_link"/>
-      <origin xyz="0 0 0.115" rpy="0 0 0"/>
+      <!-- BRAYAN (22/11/2017): Recalculo mas preciso <origin xyz="0 0 0.115" rpy="0 0 0"/> -->
+      <origin xyz="0 0 0.11363" rpy="0 0 0"/>
       <axis xyz="0 1 0"/>
       <limit effort="1000.0" lower="-1.5882496193" upper="1.5882496193" velocity="0.1"/>
@@ -75,10 +75,10 @@
       <inertial>
         <mass value="8.41"/>
-        <origin xyz="0 -0.0632 0" rpy="0 0 0"/>
+        <origin xyz="0 0 0" rpy="0 0 0"/>
         <inertia ixx="0.177079"  ixy="0.000257"  ixz="0.000005" iyy="0.018440" iyz="0.000005" izz="0.173903"/>
       </inertial>
       <visual>
         <geometry>
-          <mesh filename="package://aurobot_description/meshes/pa10-green/shoulder/S3.dae" />
+          <mesh filename="package://aurobot_description/meshes/pa10-green/shoulder/pa10_02.stl"/>
         </geometry>
         <material name="blue"/>
@@ -86,5 +86,5 @@
       <collision>
         <geometry>
-          <mesh filename="package://aurobot_description/meshes/pa10-green/shoulder/S3.stl" />
+          <mesh filename="package://aurobot_description/meshes/pa10-green/shoulder/pa10_02.stl"/>
         </geometry>
       </collision>
@@ -94,5 +94,6 @@
       <child link="${child}"/>
       <axis xyz="0 0 1"/>
-      <origin xyz="0 0 0.325" rpy="0 0 0"/>
+      <!-- BRAYAN (22/11/2017): Recalculo mas preciso <origin xyz="0 0 0.325" rpy="0 0 0"/> -->
+      <origin xyz="0 0 0.31422" rpy="0 0 0"/>
       <limit effort="1000.0" lower="-3.0368728985" upper="3.0368728985" velocity="0.2"/>
       <cfm>0.7</cfm>

File: aurobot_description/urdf/pa10-green/upper_arm/upper_arm.urdf.xacro (robot description, xacro)
@@ -11,23 +11,22 @@
   <xacro:include filename="$(find aurobot_description)/urdf/common.xacro"/>
   <!-- ============================   Upper Arm   ============================ -->
+  <!-- BRAYAN (22/11/2017): Dejamos origin a 0,0,0 en todo lo que no sea joint -->
   <xacro:macro name="pa10_green_upper_arm" params="child">
     <!-- E1: Elbow flex -->
     <link name="pa10_green_elbow_flex_link">
       <inertial>
-        <origin xyz="0 0 0.47" rpy="0 0 0"/>
         <mass value="3.51"/>
+        <origin xyz="0 0 0" rpy="0 0 0"/>
         <inertia ixx="0.032979"  ixy="0.000005"  ixz="0.000002" iyy="0.017031" iyz="0.000027" izz="0.022417"/>
       </inertial>
       <visual>
-        <origin xyz="0 0 0.125" rpy="0 0 0"/>
         <geometry>
-          <mesh filename="package://aurobot_description/meshes/pa10-green/upper_arm/E1.dae"/>
+          <mesh filename="package://aurobot_description/meshes/pa10-green/upper_arm/pa10_03.stl"/>
         </geometry>
         <material name="green"/>
       </visual>
       <collision>
-        <origin xyz="0 0 0.125" rpy="0 0 0"/>
         <geometry>
-          <mesh filename="package://aurobot_description/meshes/pa10-green/upper_arm/E1.stl"/>
+          <mesh filename="package://aurobot_description/meshes/pa10-green/upper_arm/pa10_03.stl"/>
         </geometry>
       </collision>
@@ -36,5 +35,6 @@
       <parent link="pa10_green_elbow_flex_link"/>
       <child link="pa10_green_forearm_roll_link"/>
-      <origin xyz="0 0 0.125" rpy="0 0 0"/>
+      <!-- BRAYAN (22/11/2017): Recalculo mas preciso <origin xyz="0 0 0.125" rpy="0 0 0"/> -->
+      <origin xyz="0 0 0.13578" rpy="0 0 0"/>
       <axis xyz="0 1 0"/>
       <limit effort="1000.0" lower="-2.3911010752" upper="2.3911010752" velocity="0.2"/>
@@ -45,11 +45,12 @@
     <link name="pa10_green_forearm_roll_link">
       <inertial>
-        <origin xyz="0 -0.046 0" rpy="0 0 0"/>
         <mass value="4.31"/>
+        <origin xyz="0 0 0" rpy="0 0 0"/>
         <inertia ixx="0.051762"  ixy="-0.000577"  ixz="0.000005" iyy="0.006329" iyz="0.000005" izz="0.051407"/>
       </inertial>
       <visual>
         <geometry>
-          <mesh filename="package://aurobot_description/meshes/pa10-green/upper_arm/E2.dae"/>
+          <!-- BRAYAN (22/11/2017): Escalamos esta pieza que en el STL mide 289.6 y en la realidad ronda 293.02 -->
+          <mesh filename="package://aurobot_description/meshes/pa10-green/upper_arm/pa10_04.stl" scale="1 1 1.1"/>
         </geometry>
         <material name="blue"/>
@@ -57,5 +58,5 @@
       <collision>
         <geometry>
-          <mesh filename="package://aurobot_description/meshes/pa10-green/upper_arm/E2.stl"/>
+          <mesh filename="package://aurobot_description/meshes/pa10-green/upper_arm/pa10_04.stl" scale="1 1 1.1"/>
         </geometry>
       </collision>
@@ -65,5 +66,6 @@
       <child link="${child}"/>
       <axis xyz="0 0 1"/>
-      <origin xyz="0 0 0.450" rpy="0 0 0"/>
+      <!-- BRAYAN (22/11/2017): Recalculo mas preciso <origin xyz="0 0 0.450" rpy="0 0 0"/> -->
+      <origin xyz="0 0 0.26357" rpy="0 0 0"/>
       <!-- BRAYAN (13/07/2017): gran cambio en lower y upper, casi el doble hemos puesto -->
       <limit effort="1000.0" lower="-4.4505895926" upper="4.4505895926" velocity="0.628"/>

File: aurobot_description/urdf/robot-base/trunk/trunk.urdf.xacro (robot description, xacro)
@@ -35,4 +35,14 @@
       <origin xyz="0 0.13790 1.22809" rpy="0 1.0471975512 1.5707963268"/>
     </joint>
+    <joint name="trunk_cone_joint" type="fixed">
+      <parent link="trunk_link"/>
+      <child link="cone_trunk_link"/>
+      <origin xyz="0 0 0" rpy="0 0 0"/>
+    </joint>
+    <joint name="trunk_cone2_joint" type="fixed">
+      <parent link="trunk_link"/>
+      <child link="cone2_trunk_link"/>
+      <origin xyz="0 0 0" rpy="0 0 0"/>
+    </joint>
     <joint name="trunk_head_joint" type="fixed">
       <parent link="trunk_link"/>
@@ -43,11 +53,10 @@
         Tiene en Roll (X) 112.4 negativos.
         Tiene en Pitch (Y) 0.
-        Tiene en Yaw (Z) unos 175.7 grados de desviacion -->
-      <origin xyz="0.778 1.548 1.742" rpy="-1.9634954085 0 3.0665434958"/>
-      <!--
-        Nueva prueba (19/07/2017):
-        Tiene en Roll (X) 112 negativos.
-        Tiene en Yaw (Z) unos 176.2 grados de desviacion -->
-      <!-- <origin xyz="0.775 1.537 1.735" rpy="-1.9547687622 0 3.075270142"/> -->
+        Tiene en Yaw (Z) unos 175.7 grados de desviacion
+      <origin xyz="0.778 1.548 1.742" rpy="-1.9634954085 0 3.0665434958"/>-->
+      <!-- BRAYAN (17/11/2017): posicion por calibracion de Matlab del RGB. Original:
+      <origin xyz="0.849607606 1.452407489 1.611743891" rpy="-1.9778528 -0.0034288 -3.1153181"/>
+       -->
+      <origin xyz="0.825607606 1.532407489 1.751743891" rpy="-1.9778528 -0.0034288 -3.1153181"/>
     </joint>
     <joint name="trunk_right_joint" type="fixed">

Commit message: NEW CALIBRATED POSITION. The camera has been recalibrated and the PA10 model has been modified to match the real robot (real links and joints, as well as visually positioned similarly to the real roboot through the camera)

File: aurobot_description/robots/aurobot_shadow.urdf.xacro (robot description, xacro)
@@ -127,6 +127,6 @@
   <link name="l_jr3_link">
     <inertial>
-      <origin xyz="0 0 0" rpy="0 0 0"/>
       <mass value="0.40"/>
+      <origin xyz="0 0 0" rpy="0 0 0"/>
       <inertia ixx="0.012500"  ixy="0.000005"  ixz="0.000005" iyy="0.011431" iyz="0.000005" izz="0.012500"/>
     </inertial>
@@ -146,4 +146,32 @@
   <joint name="l_jr3_joint" type="fixed">
     <parent link="l_jr3_link"/>
+    <child link="l_jr3_end_link"/>
+      <!-- BRAYAN (12/07/2017): Medimos y no tiene 10cm, son 4.7cm placa + jr3 + placa
+       <origin xyz="0 0 0.1" rpy="0 0 3.1415926536"/> -->
+      <!-- BRAYAN (22/11/2017): Realmente son 4cm, porque 0.7cm primeros son de PA10
+       <origin xyz="0 0 0.047" rpy="0 0 3.1415926536"/> -->
+    <origin xyz="0 0 0.04042" rpy="0 0 3.1415926536"/>
+  </joint>
+  <link name="l_jr3_end_link">
+    <inertial>
+      <mass value="0.40"/>
+      <origin xyz="0 0 0" rpy="0 0 0"/>
+      <inertia ixx="0.012500"  ixy="0.000005"  ixz="0.000005" iyy="0.011431" iyz="0.000005" izz="0.012500"/>
+    </inertial>
+    <visual>
+      <geometry>
+        <!-- BRAYAN (22/11/2017): Escalamos esta pieza que en el STL mide menos de la realidad -->
+        <mesh filename="package://aurobot_description/meshes/jr3/jr3.stl"/>
+      </geometry>
+      <material name="grey"/>
+    </visual>
+    <collision>
+      <geometry>
+        <mesh filename="package://aurobot_description/meshes/jr3/jr3.stl"/>
+      </geometry>
+    </collision>
+  </link>
+  <joint name="l_jr3_end_joint" type="fixed">
+    <parent link="l_jr3_end_link"/>
     <child link="l_allegro_base_link"/>
       <!-- BRAYAN (12/07/2017): Medimos y no tiene 10cm, son 4.7cm placa + jr3 + placa
@@ -151,5 +179,5 @@
       <!-- BRAYAN (22/11/2017): Realmente son 4cm, porque 0.7cm primeros son de PA10
        <origin xyz="0 0 0.047" rpy="0 0 3.1415926536"/> -->
-    <origin xyz="0 0 0.04042" rpy="0 0 3.1415926536"/>
+    <origin xyz="0 0 0.1001" rpy="0 0 0"/>
   </joint>
   <!-- Allegro left hand -->

File: aurobot_description/urdf/hand/allegro/allegro_left.urdf.xacro (robot description, xacro)
@@ -371,5 +371,4 @@
     <link name="l_allegro_base_link">
       <inertial> <!-- BRAYAN (03/07/2017): Changed to be equal to those on the allegro ros package -->
-          <!-- BRAYAN (22/11/2017): quitamos este desplazamiento del origin <origin xyz="0 0 ${base_link_z/2}" rpy="0 0 0"/>-->
           <origin xyz="0 0 ${base_link_z/2}" rpy="0 0 0"/>
           <mass value="0.4154"/>

File: aurobot_description/urdf/robot-base/trunk/trunk.urdf.xacro (robot description, xacro)
@@ -58,5 +58,5 @@
       <origin xyz="0.849607606 1.452407489 1.611743891" rpy="-1.9778528 -0.0034288 -3.1153181"/>
        -->
-      <origin xyz="0.825607606 1.532407489 1.751743891" rpy="-1.9778528 -0.0034288 -3.1153181"/>
+      <origin xyz="0.825607606 1.55407489 1.751743891" rpy="-1.9778528 -0.0034288 -3.1153181"/>
     </joint>
     <joint name="trunk_right_joint" type="fixed">
