Commit message: Readjusted the camera location. realsese_to_world now reads point clouds from the new my_sr300 node.

File: aurobot_description/robots/aurobot_shadow.urdf.xacro (robot description, xacro)
@@ -44,56 +44,4 @@
   <xacro:trunk left_child="pa10_green_shoulder_roll_link"
     head_child="head_link" right_child="pa10_blue_shoulder_roll_link"/>
-  <!-- Cono Pecho -->
-  <link name="cone_trunk_link">
-    <inertial>
-      <origin xyz="0.27501 0.0 1.328" rpy="0 ${pi/2} 0 "/>
-      <mass value="1"/>
-      <inertia
-        ixx="1.0" ixy="0.0" ixz="0.0"
-        iyy="1.0" iyz="0.0"
-        izz="1.0"/>
-    </inertial>
-    <visual>
-      <origin xyz="0.27501 0.0 1.328" rpy="0 ${pi/2} 0"/>
-      <geometry>
-        <cylinder radius="0.045" length="0.25"/>
-      </geometry>
-      <material name="Cyan">
-        <color rgba="0 1.0 1.0 0.5"/>
-      </material>
-    </visual>
-    <collision>
-      <origin xyz="0.27501 0.0 1.328" rpy="0 ${pi/2} 0"/>
-      <geometry>
-        <cylinder radius="0.045" length="0.25"/>
-      </geometry>
-    </collision>
-  </link>
-  <!-- Cono2 Pecho -->
-  <link name="cone2_trunk_link">
-    <inertial>
-      <origin xyz="0.550 0.105 1.3225" rpy="0 0 0 "/>
-      <mass value="1"/>
-      <inertia
-        ixx="1.0" ixy="0.0" ixz="0.0"
-        iyy="1.0" iyz="0.0"
-        izz="1.0"/>
-    </inertial>
-    <visual>
-      <origin xyz="0.550 0.105 1.3225" rpy="0 0 0"/>
-      <geometry>
-        <cylinder radius="0.045" length="0.25"/>
-      </geometry>
-      <material name="Cyan">
-        <color rgba="0 1.0 1.0 0.3"/>
-      </material>
-    </visual>
-    <collision>
-      <origin xyz="0.550 0.105 1.3225" rpy="0 0 0"/>
-      <geometry>
-        <cylinder radius="0.045" length="0.25"/>
-      </geometry>
-    </collision>
-  </link>
   <!-- Head -->
   <link name="head_link">
@@ -153,4 +101,5 @@
     <origin xyz="0 0 0.04042" rpy="0 0 3.1415926536"/>
   </joint>
+  <!-- BRAYAN (23/11/2017): se anyade para desplazar el visual de la mano Allegro y hacerlo coincidir con el real  -->
   <link name="l_jr3_end_link">
     <inertial>
@@ -214,12 +163,3 @@
   <!-- instantiate the hand -->
   <xacro:shadowhand lf="true" muscletrans="false" muscle="false" bio="false" bt_sp="false" ubi="false" eli="false" reflect="1.0" prefix="" />
-  <!-- virtual link for grasping
-  <joint name="hand_to_grasp" type="prismatic">
-      <parent link="palm" />
-      <child link="grasp_center" />
-      <origin xyz="0.0 -0.08 0.09" rpy="0.0 0.0 0.0" />
-      <axis xyz="0 -1 0" />
-      <limit lower="-0.08" upper="0.08" effort="30" velocity="2.0" />
-    </joint>
-  <link name="grasp_center"/>-->
 </robot>

File: aurobot_description/urdf/robot-base/trunk/trunk.urdf.xacro (robot description, xacro)
@@ -35,14 +35,4 @@
       <origin xyz="0 0.13790 1.22809" rpy="0 1.0471975512 1.5707963268"/>
     </joint>
-    <joint name="trunk_cone_joint" type="fixed">
-      <parent link="trunk_link"/>
-      <child link="cone_trunk_link"/>
-      <origin xyz="0 0 0" rpy="0 0 0"/>
-    </joint>
-    <joint name="trunk_cone2_joint" type="fixed">
-      <parent link="trunk_link"/>
-      <child link="cone2_trunk_link"/>
-      <origin xyz="0 0 0" rpy="0 0 0"/>
-    </joint>
     <joint name="trunk_head_joint" type="fixed">
       <parent link="trunk_link"/>
@@ -50,13 +40,8 @@
       <!-- BRAYAN (16/05/2017): Temporalmente puesto como una cabeza adelantada orientada hacia adelante -->
       <!-- <origin xyz="0.045 -0.025 1.71" rpy="-2.2689280276 0 -1.570796327"/> -->
-      <!-- BRAYAN (14/07/2017): posicion a la izquierda buena para agarres de frente.
-        Tiene en Roll (X) 112.4 negativos.
-        Tiene en Pitch (Y) 0.
-        Tiene en Yaw (Z) unos 175.7 grados de desviacion
-      <origin xyz="0.778 1.548 1.742" rpy="-1.9634954085 0 3.0665434958"/>-->
       <!-- BRAYAN (17/11/2017): posicion por calibracion de Matlab del RGB. Original:
       <origin xyz="0.849607606 1.452407489 1.611743891" rpy="-1.9778528 -0.0034288 -3.1153181"/>
-       -->
-      <origin xyz="0.825607606 1.55407489 1.751743891" rpy="-1.9778528 -0.0034288 -3.1153181"/>
+       x -0.015 y - 0.01-->
+      <origin xyz="0.810607606 1.54407489 1.751743891" rpy="-1.9778528 -0.0034288 -3.1153181"/>
     </joint>
     <joint name="trunk_right_joint" type="fixed">

Commit message: Camera position readjusted.

File: aurobot_description/robots/aurobot_shadow.urdf.xacro (robot description, xacro)
@@ -37,4 +37,31 @@
     <parent link="world"/>
     <child link="profiles_link"/>
+  </joint>
+  <!-- 2 Tables -->
+  <link name="table_link">
+    <inertial>
+      <origin xyz="0 0 0" rpy="0 0 0"/>
+      <mass value="1"/>
+      <inertia
+        ixx="1.0" ixy="0.0" ixz="0.0"
+        iyy="1.0" iyz="0.0"
+        izz="1.0"/>
+    </inertial>
+    <visual>
+      <geometry>
+        <box size="${0.395*2} 0.800 0.016"/>
+      </geometry>
+      <material name="orange"/>
+    </visual>
+    <collision>
+      <geometry>
+        <box size="${0.395*2} 0.800 0.016"/>
+      </geometry>
+    </collision>
+  </link>
+  <joint name="table_joint" type="fixed">
+    <parent link="world"/>
+    <child link="table_link"/>
+    <origin xyz="0.761 0.2285 1.183" rpy="0 0 0"/>
   </joint>
   <!-- Add the base -->

File: aurobot_description/urdf/robot-base/trunk/trunk.urdf.xacro (robot description, xacro)
@@ -40,8 +40,13 @@
       <!-- BRAYAN (16/05/2017): Temporalmente puesto como una cabeza adelantada orientada hacia adelante -->
       <!-- <origin xyz="0.045 -0.025 1.71" rpy="-2.2689280276 0 -1.570796327"/> -->
-      <!-- BRAYAN (17/11/2017): posicion por calibracion de Matlab del RGB. Original:
+      <!-- BRAYAN (17/11/2017): posicion por calibracion de Matlab del RGB.
+      Original:
       <origin xyz="0.849607606 1.452407489 1.611743891" rpy="-1.9778528 -0.0034288 -3.1153181"/>
-       x -0.015 y - 0.01-->
+      Bueno (sin la mesa):
       <origin xyz="0.810607606 1.54407489 1.751743891" rpy="-1.9778528 -0.0034288 -3.1153181"/>
+      Bueno (con mesa):
+      <origin xyz="0.830607606 1.53007489 1.751743891" rpy="-1.9778528 -0.0034288 -3.1353181"/>
+      -->
+      <origin xyz="0.830607606 1.53007489 1.765743891" rpy="-1.9908528 0.0044288 -3.1353181"/>
     </joint>
     <joint name="trunk_right_joint" type="fixed">

Commit message: Recalibration of the camera. Almost there (before x-mas)

File: aurobot_description/robots/aurobot_shadow.urdf.xacro (robot description, xacro)
@@ -50,5 +50,5 @@
     <visual>
       <geometry>
-        <box size="${0.395*2} 0.800 0.016"/>
+        <box size="0.794 0.800 0.016"/>
       </geometry>
       <material name="orange"/>
@@ -56,5 +56,5 @@
     <collision>
       <geometry>
-        <box size="${0.395*2} 0.800 0.016"/>
+        <box size="0.794 0.800 0.016"/>
       </geometry>
     </collision>
@@ -63,5 +63,13 @@
     <parent link="world"/>
     <child link="table_link"/>
+    <!-- BRAYAN (19/12/2017): tras descalibrado de camara y mesa.
+    Anterior:
     <origin xyz="0.761 0.2285 1.183" rpy="0 0 0"/>
+    Bien medido:
+    <origin xyz="0.759 0.210 1.180" rpy="0 0 0"/>
+    Esta es buena para agarres frontales pero falla hacia abajo
+    <origin xyz="0.759 0.2485 1.147" rpy="0 0 0"/>
+    -->
+    <origin xyz="0.759 0.210 1.180" rpy="0 0 0"/>
   </joint>
   <!-- Add the base -->

File: aurobot_description/urdf/robot-base/trunk/trunk.urdf.xacro (robot description, xacro)
@@ -41,12 +41,16 @@
       <!-- <origin xyz="0.045 -0.025 1.71" rpy="-2.2689280276 0 -1.570796327"/> -->
       <!-- BRAYAN (17/11/2017): posicion por calibracion de Matlab del RGB.
-      Original:
-      <origin xyz="0.849607606 1.452407489 1.611743891" rpy="-1.9778528 -0.0034288 -3.1153181"/>
-      Bueno (sin la mesa):
-      <origin xyz="0.810607606 1.54407489 1.751743891" rpy="-1.9778528 -0.0034288 -3.1153181"/>
       Bueno (con mesa):
-      <origin xyz="0.830607606 1.53007489 1.751743891" rpy="-1.9778528 -0.0034288 -3.1353181"/>
+      <origin xyz="0.830607606 1.53007489 1.765743891" rpy="-1.9908528 0.0044288 -3.1353181"/>
+      new-my-checkers: [ x: -2.743256, y: 0.0229434, z: -0.0118721 ]
+      <origin xyz="0.830607606 1.53007489 1.7083008379" rpy="-1.957857825 0.00229434 -3.1297206"/>
+      new-my-checkers-v2: [ x: -2.7073592, y: -0.0542398, z: -1.5664367 ]
+      <origin xyz="0.825607606 1.54007489 1.745743891" rpy="-1.985961037 0.00542398 -3.127233027"/>
+      new-my-checkers-v3: [ x: -2.693058, y: -0.0482789, z: -3.1355064 ]
+      <origin xyz="0.849 1.48349 1.71034" rpy="-2.693058 -0.0482789 -3.1355064"/>
+      Esta es buena para agarres frontales pero falla hacia abajo
+      <origin xyz="0.820 1.54049 1.73034" rpy="-1.9945 0.00562789 -3.1305064"/>
       -->
-      <origin xyz="0.830607606 1.53007489 1.765743891" rpy="-1.9908528 0.0044288 -3.1353181"/>
+      <origin xyz="0.820 1.54049 1.73034" rpy="-1.9645 0.00562789 -3.1105064"/>
     </joint>
     <joint name="trunk_right_joint" type="fixed">

Commit message: Recalibrated the camera position. Not as good as the last time, but acceptable.

File: aurobot_description/robots/aurobot_shadow.urdf.xacro (robot description, xacro)
@@ -68,8 +68,8 @@
     Bien medido:
     <origin xyz="0.759 0.210 1.180" rpy="0 0 0"/>
-    Esta es buena para agarres frontales pero falla hacia abajo
-    <origin xyz="0.759 0.2485 1.147" rpy="0 0 0"/>
+    Esta es buena para agarres frontales pero falla hacia abajo:
+    <origin xyz="0.759 0.2385 1.149" rpy="0 0 0"/>
     -->
-    <origin xyz="0.759 0.210 1.180" rpy="0 0 0"/>
+    <origin xyz="0.759 0.2385 1.149" rpy="0 0 0"/>
   </joint>
   <!-- Add the base -->

File: aurobot_description/urdf/robot-base/trunk/trunk.urdf.xacro (robot description, xacro)
@@ -43,14 +43,12 @@
       Bueno (con mesa):
       <origin xyz="0.830607606 1.53007489 1.765743891" rpy="-1.9908528 0.0044288 -3.1353181"/>
-      new-my-checkers: [ x: -2.743256, y: 0.0229434, z: -0.0118721 ]
-      <origin xyz="0.830607606 1.53007489 1.7083008379" rpy="-1.957857825 0.00229434 -3.1297206"/>
-      new-my-checkers-v2: [ x: -2.7073592, y: -0.0542398, z: -1.5664367 ]
-      <origin xyz="0.825607606 1.54007489 1.745743891" rpy="-1.985961037 0.00542398 -3.127233027"/>
-      new-my-checkers-v3: [ x: -2.693058, y: -0.0482789, z: -3.1355064 ]
-      <origin xyz="0.849 1.48349 1.71034" rpy="-2.693058 -0.0482789 -3.1355064"/>
+      new-my-checkers (3): [ x: -2.693058, y: -0.0482789, z: -3.1355064 ]
+      new-my-checkers-2: [ x: -2.7024739, y: 0.0619603, z: -3.1274342 ]
+      <origin xyz="0.830 1.530 1.765" rpy="-1.917075737 0.0619603 -3.1274342"/>
+      BRAYAN (10/01/2018):
       Esta es buena para agarres frontales pero falla hacia abajo
-      <origin xyz="0.820 1.54049 1.73034" rpy="-1.9945 0.00562789 -3.1305064"/>
+      <origin xyz="0.820 1.54549 1.72834" rpy="-1.9895 0.00500789 -3.1290064"/>
       -->
-      <origin xyz="0.820 1.54049 1.73034" rpy="-1.9645 0.00562789 -3.1105064"/>
+      <origin xyz="0.820 1.54549 1.72834" rpy="-1.9895 0.00500789 -3.1290064"/>
     </joint>
     <joint name="trunk_right_joint" type="fixed">

Commit message: Update control grasp loop. The newer loop lets the user repeat the planning in case MoveIt! has found a strange trajectory.

File: aurobot_description/robots/aurobot_shadow.urdf.xacro (robot description, xacro)
@@ -167,10 +167,11 @@
   <!-- Allegro left hand -->
   <xacro:allegro_left_hand/>
+  <link name="pa10_blue_shoulder_roll_link" />
   <!-- Add the right PA10 -->
-  <xacro:pa10_blue_shoulder child="pa10_blue_elbow_flex_link"/>
+  <!-- <xacro:pa10_blue_shoulder child="pa10_blue_elbow_flex_link"/>
   <xacro:pa10_blue_upper_arm child="pa10_blue_wrist_flex_link"/>
-  <xacro:pa10_blue_forearm child="r_jr3_link"/>
+  <xacro:pa10_blue_forearm child="r_jr3_link"/> -->
   <!-- JR3 right -->
-  <link name="r_jr3_link">
+  <!-- <link name="r_jr3_link">
     <inertial>
       <origin xyz="0 0 0" rpy="0 0 0"/>
@@ -189,12 +190,12 @@
       </geometry>
     </collision>
-  </link>
+  </link> -->
   <!-- attach the hand to the arm -->
-  <joint name="r_jr3_joint" type="fixed">
+  <!-- <joint name="r_jr3_joint" type="fixed">
     <parent link="r_jr3_link" />
     <child link = "forearm" />
     <origin xyz="0 0 0" rpy="0 0 ${pi/2.0}"/>
-  </joint>
+  </joint> -->
   <!-- instantiate the hand -->
-  <xacro:shadowhand lf="true" muscletrans="false" muscle="false" bio="false" bt_sp="false" ubi="false" eli="false" reflect="1.0" prefix="" />
+  <!-- <xacro:shadowhand lf="true" muscletrans="false" muscle="false" bio="false" bt_sp="false" ubi="false" eli="false" reflect="1.0" prefix="" /> -->
 </robot>

File: aurobot_description/urdf/robot-base/trunk/trunk.urdf.xacro (robot description, xacro)
@@ -50,5 +50,5 @@
       <origin xyz="0.820 1.54549 1.72834" rpy="-1.9895 0.00500789 -3.1290064"/>
       -->
-      <origin xyz="0.820 1.54549 1.72834" rpy="-1.9895 0.00500789 -3.1290064"/>
+      <origin xyz="0.807 1.51849 1.74534" rpy="-2.0375 0.0150079 -3.12501"/>
     </joint>
     <joint name="trunk_right_joint" type="fixed">
