Commit message: Add 3D printed coupling (right arm).

File: aurobot_description/robots/aurobot_right.urdf.xacro (robot description, xacro)
@@ -53,12 +53,4 @@
     <parent link="world"/>
     <child link="table_link"/>
-    <!-- BRAYAN (19/12/2017): tras descalibrado de camara y mesa.
-    Anterior:
-    <origin xyz="0.761 0.2285 1.183" rpy="0 0 0"/>
-    Bien medido:
-    <origin xyz="0.759 0.210 1.180" rpy="0 0 0"/>
-    Esta es buena para agarres frontales pero falla hacia abajo:
-    <origin xyz="0.759 0.2385 1.149" rpy="0 0 0"/>
-    -->
     <origin xyz="0.759 0.2385 1.149" rpy="0 0 0"/>
   </joint>
@@ -108,5 +100,5 @@
     <visual>
       <geometry>
-      <mesh filename="package://aurobot_description/meshes/jr3/jr3.stl"/>
+        <mesh filename="package://aurobot_description/meshes/jr3/jr3.stl" scale="1 1 8"/>
       </geometry>
       <material name="grey"/>
@@ -114,5 +106,29 @@
     <collision>
       <geometry>
-        <mesh filename="package://aurobot_description/meshes/jr3/jr3.stl"/>
+        <mesh filename="package://aurobot_description/meshes/jr3/jr3.stl" scale="1 1 8"/>
+      </geometry>
+    </collision>
+  </link>
+  <joint name="coupling_joint" type="fixed">
+    <parent link="r_jr3_link"/>
+    <child link="r_coupling_link"/>
+    <origin xyz="0 0 0.051" rpy="0 0 0"/>
+  </joint>
+  <!-- Coupling -->
+  <link name="r_coupling_link">
+    <inertial>
+      <origin xyz="0 0 0" rpy="0 0 0"/>
+      <mass value="0.40"/>
+      <inertia ixx="0.012500"  ixy="0.000005"  ixz="0.000005" iyy="0.011431" iyz="0.000005" izz="0.012500"/>
+    </inertial>
+    <visual>
+      <geometry>
+        <mesh filename="package://aurobot_description/meshes/coupling/CouplingRobotic.stl" scale="0.001 0.001 0.001"/>
+      </geometry>
+      <material name="green"/>
+    </visual>
+    <collision>
+      <geometry>
+        <mesh filename="package://aurobot_description/meshes/coupling/CouplingRobotic.stl" scale="0.001 0.001 0.001"/>
       </geometry>
     </collision>

File: aurobot_description/urdf/pa10-blue/forearm/forearm.urdf.xacro (robot description, xacro)
@@ -64,5 +64,6 @@
       <parent link="pa10_blue_wrist_roll_link"/>
       <child link="${child}"/>
-      <origin xyz="0 0 0.075" rpy="0 0 0"/>
+      <!-- <origin xyz="0 0 0.075" rpy="0 0 0"/> -->
+      <origin xyz="0 0 0.0705" rpy="0 0 0"/>
       <axis xyz="0 0 1"/>
       <limit effort="1000.0" lower="-2.878" upper="2.878" velocity="0.628"/>
