Commit message: Update the name of the left camera link in the URDFs and the grasping scripts.

File: aurobot_description/robots/aurobot_left.urdf.xacro (robot description, xacro)
@@ -69,8 +69,7 @@
   <xacro:base child="bearing_under_link"/>
   <xacro:bearing child="trunk_link"/>
-  <xacro:trunk left_child="pa10_green_shoulder_roll_link"
-    head_child="head_link" right_child="pa10_blue_shoulder_roll_link"/>
-  <!-- Head -->
-  <link name="head_link">
+  <xacro:trunk/>
+  <!-- Left camera -->
+  <link name="left_camera_link">
     <inertial>
       <origin xyz="0 0 1" rpy="0 0 0"/>
@@ -95,8 +94,30 @@
     </collision>
   </link>
+  <joint name="left_camera_joint" type="fixed">
+    <parent link="trunk_link"/>
+    <child link="left_camera_link"/>
+    <!-- BRAYAN (16/05/2017): Temporalmente puesto como una cabeza adelantada orientada hacia adelante -->
+    <!-- <origin xyz="0.045 -0.025 1.71" rpy="-2.2689280276 0 -1.570796327"/> -->
+    <!-- BRAYAN (17/11/2017): posicion por calibracion de Matlab del RGB.
+    Bueno (con mesa):
+    <origin xyz="0.830607606 1.53007489 1.765743891" rpy="-1.9908528 0.0044288 -3.1353181"/>
+    new-my-checkers (3): [ x: -2.693058, y: -0.0482789, z: -3.1355064 ]
+    new-my-checkers-2: [ x: -2.7024739, y: 0.0619603, z: -3.1274342 ]
+    <origin xyz="0.830 1.530 1.765" rpy="-1.917075737 0.0619603 -3.1274342"/>
+    BRAYAN (10/01/2018):
+    Esta es buena para agarres frontales pero falla hacia abajo
+    <origin xyz="0.820 1.54549 1.72834" rpy="-1.9895 0.00500789 -3.1290064"/>
+    -->
+    <origin xyz="0.807 1.51849 1.74534" rpy="-2.0375 0.0150079 -3.12501"/>
+  </joint>
   <!-- Add the left PA10 -->
   <xacro:pa10_green_shoulder child="pa10_green_elbow_flex_link"/>
   <xacro:pa10_green_upper_arm child="pa10_green_wrist_flex_link"/>
   <xacro:pa10_green_forearm child="l_jr3_link"/>
+  <joint name="trunk_left_joint" type="fixed">
+    <parent link="trunk_link"/>
+    <child link="pa10_green_shoulder_roll_link"/>
+    <origin xyz="0 0.13790 1.22809" rpy="0 1.0471975512 1.5707963268"/>
+  </joint>
   <!-- JR3 left -->
   <link name="l_jr3_link">
@@ -159,4 +180,3 @@
   <!-- Allegro left hand -->
   <xacro:allegro_left_hand/>
-  <link name="pa10_blue_shoulder_roll_link" />
 </robot>

File: aurobot_description/robots/aurobot_right_robotiq.urdf.xacro (robot description, xacro)
@@ -61,10 +61,7 @@
   <xacro:base child="bearing_under_link"/>
   <xacro:bearing child="trunk_link"/>
-  <xacro:trunk left_child="pa10_green_shoulder_roll_link"
-    head_child="head_link" right_child="pa10_blue_shoulder_roll_link"/>
-  <!-- Left link -->
-  <link name="pa10_green_shoulder_roll_link" />
-  <!-- Head -->
-  <link name="head_link">
+  <xacro:trunk/>
+  <!-- Left camera -->
+  <link name="left_camera_link">
     <inertial>
       <origin xyz="0 0 1" rpy="0 0 0"/>
@@ -89,8 +86,18 @@
     </collision>
   </link>
+  <joint name="left_camera_joint" type="fixed">
+    <parent link="trunk_link"/>
+    <child link="left_camera_link"/>
+    <origin xyz="0.807 1.51849 1.74534" rpy="-2.0375 0.0150079 -3.12501"/>
+  </joint>
   <!-- Add the right PA10 -->
   <xacro:pa10_blue_shoulder child="pa10_blue_elbow_flex_link"/>
   <xacro:pa10_blue_upper_arm child="pa10_blue_wrist_flex_link"/>
   <xacro:pa10_blue_forearm child="r_jr3_link"/>
+  <joint name="trunk_right_joint" type="fixed">
+    <parent link="trunk_link"/>
+    <child link="pa10_blue_shoulder_roll_link"/>
+    <origin xyz="0 -0.13790 1.22809" rpy="0 -1.0471975512 1.5707963268"/>
+  </joint>
   <!-- JR3 right -->
   <link name="r_jr3_link">

File: aurobot_description/robots/aurobot_right_shadow.urdf.xacro (robot description, xacro)
@@ -63,10 +63,7 @@
   <xacro:base child="bearing_under_link"/>
   <xacro:bearing child="trunk_link"/>
-  <xacro:trunk left_child="pa10_green_shoulder_roll_link"
-    head_child="head_link" right_child="pa10_blue_shoulder_roll_link"/>
-  <!-- Left link -->
-  <link name="pa10_green_shoulder_roll_link" />
-  <!-- Head -->
-  <link name="head_link">
+  <xacro:trunk/>
+  <!-- Left camera -->
+  <link name="left_camera_link">
     <inertial>
       <origin xyz="0 0 1" rpy="0 0 0"/>
@@ -91,8 +88,18 @@
     </collision>
   </link>
+  <joint name="left_camera_joint" type="fixed">
+    <parent link="trunk_link"/>
+    <child link="left_camera_link"/>
+    <origin xyz="0.807 1.51849 1.74534" rpy="-2.0375 0.0150079 -3.12501"/>
+  </joint>
   <!-- Add the right PA10 -->
   <xacro:pa10_blue_shoulder child="pa10_blue_elbow_flex_link"/>
   <xacro:pa10_blue_upper_arm child="pa10_blue_wrist_flex_link"/>
   <xacro:pa10_blue_forearm child="r_jr3_link"/>
+  <joint name="trunk_right_joint" type="fixed">
+    <parent link="trunk_link"/>
+    <child link="pa10_blue_shoulder_roll_link"/>
+    <origin xyz="0 -0.13790 1.22809" rpy="0 -1.0471975512 1.5707963268"/>
+  </joint>
   <!-- JR3 right -->
   <link name="r_jr3_link">

File: aurobot_description/urdf/robot-base/trunk/trunk.urdf.xacro (robot description, xacro)
@@ -10,5 +10,5 @@
   <xacro:include filename="$(find aurobot_description)/urdf/common.xacro"/>
  <!-- ============================   Profiles   ============================ -->
-  <xacro:macro name="trunk" params="left_child head_child right_child">
+  <xacro:macro name="trunk">
     <!-- Trunk link -->
     <link name="trunk_link">
@@ -30,31 +30,4 @@
       </collision>
     </link>
-    <joint name="trunk_left_joint" type="fixed">
-      <parent link="trunk_link"/>
-      <child link="${left_child}"/>
-      <origin xyz="0 0.13790 1.22809" rpy="0 1.0471975512 1.5707963268"/>
-    </joint>
-    <joint name="trunk_head_joint" type="fixed">
-      <parent link="trunk_link"/>
-      <child link="${head_child}"/>
-      <!-- BRAYAN (16/05/2017): Temporalmente puesto como una cabeza adelantada orientada hacia adelante -->
-      <!-- <origin xyz="0.045 -0.025 1.71" rpy="-2.2689280276 0 -1.570796327"/> -->
-      <!-- BRAYAN (17/11/2017): posicion por calibracion de Matlab del RGB.
-      Bueno (con mesa):
-      <origin xyz="0.830607606 1.53007489 1.765743891" rpy="-1.9908528 0.0044288 -3.1353181"/>
-      new-my-checkers (3): [ x: -2.693058, y: -0.0482789, z: -3.1355064 ]
-      new-my-checkers-2: [ x: -2.7024739, y: 0.0619603, z: -3.1274342 ]
-      <origin xyz="0.830 1.530 1.765" rpy="-1.917075737 0.0619603 -3.1274342"/>
-      BRAYAN (10/01/2018):
-      Esta es buena para agarres frontales pero falla hacia abajo
-      <origin xyz="0.820 1.54549 1.72834" rpy="-1.9895 0.00500789 -3.1290064"/>
-      -->
-      <origin xyz="0.807 1.51849 1.74534" rpy="-2.0375 0.0150079 -3.12501"/>
-    </joint>
-    <joint name="trunk_right_joint" type="fixed">
-      <parent link="trunk_link"/>
-      <child link="${right_child}"/>
-      <origin xyz="0 -0.13790 1.22809" rpy="0 -1.0471975512 1.5707963268"/>
-    </joint>
     <!-- extensions   -->
     <xacro:trunk_gazebo/>
