Commit message: Update links and joints names related to the Shadow so they are equivalent to those in the shadow workspace.

File: aurobot_description/robots/aurobot_right_shadow.urdf.xacro (robot description, xacro)
@@ -145,8 +145,8 @@
   <joint name="r_coupling_joint" type="fixed">
     <parent link="r_coupling_link"/>
-    <child link="forearm"/>
+    <child link="rh_forearm"/>
     <origin xyz="0 0 0.0025" rpy="0 0 ${pi/2.0}"/>
   </joint>
   <!-- instantiate the hand -->
-  <xacro:shadowhand lf="true" muscletrans="false" muscle="false" bio="false" bt_sp="false" ubi="false" eli="false" reflect="1.0" prefix="" />
+  <xacro:shadowhand lf="true" muscletrans="false" muscle="false" bio="false" bt_sp="true" ubi="false" eli="false" reflect="1.0" prefix="rh_" />
 </robot>

Commit message: Add calibrated position of the camera (top).

File: aurobot_description/robots/aurobot_right_shadow.urdf.xacro (robot description, xacro)
@@ -64,8 +64,8 @@
   <xacro:bearing child="trunk_link"/>
   <xacro:trunk/>
-  <!-- Left camera -->
-  <link name="left_camera_link">
+  <!-- Top camera -->
+  <link name="top_camera_link">
     <inertial>
-      <origin xyz="0 0 1" rpy="0 0 0"/>
+      <origin xyz="0 0 0" rpy="0 0 0"/>
       <mass value="1"/>
       <inertia
@@ -79,5 +79,5 @@
         <box size="0.025 0.025 0.025"/>
       </geometry>
-      <material name="black"/>
+      <material name="orange"/>
     </visual>
     <collision>
@@ -88,9 +88,9 @@
     </collision>
   </link>
-  <joint name="left_camera_joint" type="fixed">
-    <parent link="trunk_link"/>
-    <child link="left_camera_link"/>
-    <origin xyz="0.807 1.51849 1.74534" rpy="-2.0375 0.0150079 -3.12501"/>
-  </joint>
+  <joint name="top_camera_joint" type="fixed">
+    <parent link="world"/>
+    <child link="top_camera_link"/>
+    <origin xyz="0.62 -0.097 2.456" rpy="0.01 -3.18 -4.73"/>
+  </joint>-->
   <!-- Add the right PA10 -->
   <xacro:pa10_blue_shoulder child="pa10_blue_elbow_flex_link"/>

Commit message: Update top camera position after correctly checking its calibration with the real robot.

File: aurobot_description/robots/aurobot_right_shadow.urdf.xacro (robot description, xacro)
@@ -57,5 +57,5 @@
     <parent link="world"/>
     <child link="table_link"/>
-    <origin xyz="0.759 0.2385 1.149" rpy="0 0 0"/>
+    <origin xyz="0.759 0.215 1.18" rpy="0 0 0"/>
   </joint>
   <!-- Add the base -->
@@ -91,5 +91,5 @@
     <parent link="world"/>
     <child link="top_camera_link"/>
-    <origin xyz="0.62 -0.097 2.456" rpy="0.01 -3.18 -4.73"/>
+    <origin xyz="0.589 -0.117 2.486" rpy="0.03 -3.18 -4.728"/>
   </joint>-->
   <!-- Add the right PA10 -->

Commit message: New top-camera calibration.

File: aurobot_description/robots/aurobot_right_shadow.urdf.xacro (robot description, xacro)
@@ -91,5 +91,6 @@
     <parent link="world"/>
     <child link="top_camera_link"/>
-    <origin xyz="0.589 -0.117 2.486" rpy="0.03 -3.18 -4.728"/>
+    <!--<origin xyz="0.589 -0.117 2.486" rpy="0.03 -3.18 -4.728"/>-->
+    <origin xyz="0.589 -0.097 2.49" rpy="0.03 -3.16 -4.728"/>
   </joint>-->
   <!-- Add the right PA10 -->

Commit message: Add new calibration (top) and calculus for shadow pose (in develop).

File: aurobot_description/robots/aurobot_right_shadow.urdf.xacro (robot description, xacro)
@@ -92,5 +92,5 @@
     <child link="top_camera_link"/>
     <!--<origin xyz="0.589 -0.117 2.486" rpy="0.03 -3.18 -4.728"/>-->
-    <origin xyz="0.589 -0.097 2.49" rpy="0.03 -3.16 -4.728"/>
+    <origin xyz="0.589 -0.11 2.49" rpy="0.03 -3.16 -4.728"/>
   </joint>-->
   <!-- Add the right PA10 -->
