Commit message: New robot description: Shadow hand attached to the right PA10. MoveIt! is still to be configured to include it.

File: aurobot_description/urdf/hand/allegro/allegro_left.urdf.xacro (robot description, xacro)
@@ -199,5 +199,5 @@
   <!-- THREE FINGER MACRO -->
   <!-- ============================================================================= -->
-  <xacro:macro name="finger" params="finger_num offset_origin_x offset_origin_y offset_origin_z finger_angle_r">
+  <xacro:macro name="allegro_finger" params="finger_num offset_origin_x offset_origin_y offset_origin_z finger_angle_r">
     <!-- [LINK 0, 4, 8] -->
     <link name="l_allegro_link_${finger_num*4+0}">
@@ -373,5 +373,5 @@
     />
     <!-- FINGERS -->
-    <xacro:finger
+    <xacro:allegro_finger
       finger_num=     "2"
       offset_origin_x=  "${offset_origin_x_const}"
@@ -380,5 +380,5 @@
       finger_angle_r=   "-${5.0*DEG2RAD}"
     />
-    <xacro:finger
+    <xacro:allegro_finger
       finger_num=     "1"
       offset_origin_x=  "${offset_origin_x_const}"
@@ -387,5 +387,5 @@
       finger_angle_r=   "0.0"
     />
-    <xacro:finger
+    <xacro:allegro_finger
       finger_num=     "0"
       offset_origin_x=  "${offset_origin_x_const}"
