Commit message: fixing the simulated camera position to represent the real state

File: aurobot_description/urdf/robot-base/profiles/profiles.urdf.xacro (robot description, xacro)
@@ -15,5 +15,5 @@
       <inertial>
         <mass value="12.43"/>
-        <origin xyz="0 0 0" rpy="0 0 0"/>
+        <origin xyz="0 0 0.006" rpy="0 0 0"/> <!-- BRAYAN (10/07/2017): Se suma 0.006m de las patas de goma -->
         <inertia ixx="0.00"  ixy="0.00"  ixz="0.00" iyy="0.00" iyz="0.00" izz="0.00"/>
       </inertial>

File: aurobot_description/urdf/robot-base/trunk/trunk.urdf.xacro (robot description, xacro)
@@ -41,6 +41,6 @@
       -1.570796327 0 -1.570796327-->
       <!-- <origin xyz="0.045 -0.025 1.71" rpy="-2.2689280276 0 -1.570796327"/> -->
-      <!-- BRAYAN (04/07/2017): posicion a la izquierda -->
-      <origin xyz="0.69 1.366 1.765" rpy="-1.9722220548 0 3.1415926536"/>
+      <!-- BRAYAN (10/07/2017): posicion a la izquierda. Tiene rotado en Z unos 180 + 3 grados de desviacion -->
+      <origin xyz="0.717 1.5334 1.731" rpy="-1.9722220548 0 3.1590459461"/>
     </joint>
     <joint name="trunk_right_joint" type="fixed">
