Commit message: Updated the pa10 description to match the manual. Joints are now distanced from each other exactly like in the manual.

File: aurobot_description/urdf/pa10-green/forearm/forearm.urdf (copy).xacro (robot description, xacro)
@@ -15,9 +15,10 @@
     <link name="pa10_green_wrist_flex_link">
       <inertial>
-        <origin xyz="0 0 0" rpy="0 0 0"/>
+        <origin xyz="0 -0.0432 0.03" rpy="0 0 0"/>
         <mass value="3.45"/>
         <inertia ixx="0.076687"  ixy="0.000005"  ixz="0.000960" iyy="0.077392" iyz="0.000005" izz="0.006233"/>
       </inertial>
       <visual>
+        <origin xyz="0 0 0.03" rpy="0 0 0"/>
         <geometry>
           <mesh filename="package://aurobot_description/meshes/pa10-green/forearm/W1.dae"/>
@@ -26,4 +27,5 @@
       </visual>
       <collision>
+        <origin xyz="0 0 0.03" rpy="0 0 0"/>
         <geometry>
           <mesh filename="package://aurobot_description/meshes/pa10-green/forearm/W1.stl"/>
@@ -34,7 +36,7 @@
       <parent link="pa10_green_wrist_flex_link"/>
       <child link="pa10_green_wrist_roll_link"/>
-      <origin xyz="0 0 0.239" rpy="0 0 0"/>
+      <origin xyz="0 0 0.05" rpy="0 0 0"/>
       <axis xyz="0 1 0"/>
-      <limit effort="1000.0" lower="-2.8797932658" upper="2.8797932658" velocity="0.628"/>
+      <limit effort="1000.0" lower="-2.88" upper="2.88" velocity="0.628"/>
       <cfm>0.7</cfm>
     </joint>
@@ -42,9 +44,10 @@
     <link name="pa10_green_wrist_roll_link">
       <inertial>
-        <origin xyz="0 0 0" rpy="0 0 0"/>
+        <origin xyz="0 0.003 -0.0175" rpy="0 0 0"/>
         <mass value="1.46"/>
         <inertia ixx="0.012500"  ixy="0.000005"  ixz="0.000005" iyy="0.011431" iyz="0.000005" izz="0.012500"/>
       </inertial>
       <visual>
+        <origin xyz="0 0.0 -0.0175" rpy="0 0 0"/>
         <geometry>
           <mesh filename="package://aurobot_description/meshes/pa10-green/forearm/W2.dae"/>
@@ -53,4 +56,5 @@
       </visual>
       <collision>
+        <origin xyz="0 0.0 -0.0175" rpy="0 0 0"/>
         <geometry>
           <mesh filename="package://aurobot_description/meshes/pa10-green/forearm/W2.stl"/>
@@ -64,6 +68,5 @@
       <origin xyz="0 0 0.080" rpy="0 0 0"/>
       <axis xyz="0 0 1"/>
-      <!-- BRAYAN (13/07/2017): gran cambio en lower y upper, casi el doble hemos puesto -->
-      <limit effort="1000.0" lower="-6.2831853072" upper="6.2831853072" velocity="0.628"/>
+      <limit effort="1000.0" lower="-2.0" upper="2.28" velocity="0.628"/>
       <cfm>0.7</cfm>
     </joint>

File: aurobot_description/urdf/pa10-green/shoulder/shoulder.urdf (another copy).xacro (robot description, xacro)
@@ -35,5 +35,5 @@
       <child link="pa10_green_shoulder_lift_link"/>
       <!-- BRAYAN (12/07/2017): Segun el manual nos sobra 0.001 <origin xyz="0 0 0.201" rpy="0 0 0"/> -->
-      <origin xyz="0 0 0.199" rpy="0 0 0"/>
+      <origin xyz="0 0 0.20" rpy="0 0 0"/>
       <axis xyz="0 0 1"/>
       <limit effort="1000.0" lower="-3.089232776" upper="3.089232776" velocity="0.1"/>
@@ -45,8 +45,9 @@
       <inertial>
         <mass value="9.78"/>
-        <origin xyz="0 0 0" rpy="0 0 0"/>
+        <origin xyz="0 0 0.115" rpy="0 0 0"/>
         <inertia ixx="0.110697"  ixy="0.000005"  ixz="0.000345" iyy="0.084268" iyz="0.000518" izz="0.054080"/>
       </inertial>
       <visual>
+        <origin xyz="0 0 0.115" rpy="0 0 0"/>
         <geometry>
           <mesh filename="package://aurobot_description/meshes/pa10-green/shoulder/S2.dae"/>
@@ -55,4 +56,5 @@
       </visual>
       <collision>
+        <origin xyz="0 0 0.115" rpy="0 0 0"/>
         <geometry>
           <mesh filename="package://aurobot_description/meshes/pa10-green/shoulder/S2.stl" />
@@ -63,5 +65,5 @@
       <parent link="pa10_green_shoulder_lift_link"/>
       <child link="pa10_green_upper_arm_roll_link"/>
-      <origin xyz="0 0 0.116" rpy="0 0 0"/>
+      <origin xyz="0 0 0.115" rpy="0 0 0"/>
       <axis xyz="0 1 0"/>
       <limit effort="1000.0" lower="-1.5882496193" upper="1.5882496193" velocity="0.1"/>
@@ -73,5 +75,5 @@
       <inertial>
         <mass value="8.41"/>
-        <origin xyz="0 0 0" rpy="0 0 0"/>
+        <origin xyz="0 -0.0632 0" rpy="0 0 0"/>
         <inertia ixx="0.177079"  ixy="0.000257"  ixz="0.000005" iyy="0.018440" iyz="0.000005" izz="0.173903"/>
       </inertial>
@@ -92,5 +94,5 @@
       <child link="${child}"/>
       <axis xyz="0 0 1"/>
-      <origin xyz="0 0 0.186" rpy="0 0 0"/>
+      <origin xyz="0 0 0.325" rpy="0 0 0"/>
       <limit effort="1000.0" lower="-3.0368728985" upper="3.0368728985" velocity="0.2"/>
       <cfm>0.7</cfm>

File: aurobot_description/urdf/pa10-green/shoulder/shoulder.urdf (copy).xacro (robot description, xacro)
@@ -35,7 +35,7 @@
       <child link="pa10_green_shoulder_lift_link"/>
       <!-- BRAYAN (12/07/2017): Segun el manual nos sobra 0.001 <origin xyz="0 0 0.201" rpy="0 0 0"/> -->
-      <origin xyz="0 0 0.199" rpy="0 0 0"/>
+      <origin xyz="0 0 0.20" rpy="0 0 0"/>
       <axis xyz="0 0 1"/>
-      <limit effort="1000.0" lower="-3.089232776" upper="3.089232776" velocity="0.1"/>
+      <limit effort="1000.0" lower="-3.09" upper="3.09" velocity="0.1"/>
       <cfm>0.7</cfm>
       <damping>10.0</damping>
@@ -45,8 +45,9 @@
       <inertial>
         <mass value="9.78"/>
-        <origin xyz="0 0 0" rpy="0 0 0"/>
+        <origin xyz="0 0 0.115" rpy="0 0 0"/>
         <inertia ixx="0.110697"  ixy="0.000005"  ixz="0.000345" iyy="0.084268" iyz="0.000518" izz="0.054080"/>
       </inertial>
       <visual>
+        <origin xyz="0 0 0.115" rpy="0 0 0"/>
         <geometry>
           <mesh filename="package://aurobot_description/meshes/pa10-green/shoulder/S2.dae"/>
@@ -55,4 +56,5 @@
       </visual>
       <collision>
+        <origin xyz="0 0 0.115" rpy="0 0 0"/>
         <geometry>
           <mesh filename="package://aurobot_description/meshes/pa10-green/shoulder/S2.stl" />
@@ -63,7 +65,7 @@
       <parent link="pa10_green_shoulder_lift_link"/>
       <child link="pa10_green_upper_arm_roll_link"/>
-      <origin xyz="0 0 0.116" rpy="0 0 0"/>
+      <origin xyz="0 0 0.115" rpy="0 0 0"/>
       <axis xyz="0 1 0"/>
-      <limit effort="1000.0" lower="-1.5882496193" upper="1.5882496193" velocity="0.1"/>
+      <limit effort="1000.0" lower="-1.59" upper="1.59" velocity="0.1"/>
       <cfm>0.7</cfm>
       <damping>10.0</damping>
@@ -73,5 +75,5 @@
       <inertial>
         <mass value="8.41"/>
-        <origin xyz="0 0 0" rpy="0 0 0"/>
+        <origin xyz="0 -0.0632 0" rpy="0 0 0"/>
         <inertia ixx="0.177079"  ixy="0.000257"  ixz="0.000005" iyy="0.018440" iyz="0.000005" izz="0.173903"/>
       </inertial>
@@ -92,6 +94,6 @@
       <child link="${child}"/>
       <axis xyz="0 0 1"/>
-      <origin xyz="0 0 0.186" rpy="0 0 0"/>
-      <limit effort="1000.0" lower="-3.0368728985" upper="3.0368728985" velocity="0.2"/>
+      <origin xyz="0 0 0.325" rpy="0 0 0"/>
+      <limit effort="1000.0" lower="-3.04" upper="3.04" velocity="0.2"/>
       <cfm>0.7</cfm>
       <damping>10.0</damping>

File: aurobot_description/urdf/pa10-green/upper_arm/upper_arm.urdf (copy).xacro (robot description, xacro)
@@ -15,9 +15,10 @@
     <link name="pa10_green_elbow_flex_link">
       <inertial>
-        <origin xyz="0 0 0" rpy="0 0 0"/>
+        <origin xyz="0 0 0.47" rpy="0 0 0"/>
         <mass value="3.51"/>
         <inertia ixx="0.032979"  ixy="0.000005"  ixz="0.000002" iyy="0.017031" iyz="0.000027" izz="0.022417"/>
       </inertial>
       <visual>
+        <origin xyz="0 0 0.125" rpy="0 0 0"/>
         <geometry>
           <mesh filename="package://aurobot_description/meshes/pa10-green/upper_arm/E1.dae"/>
@@ -26,4 +27,5 @@
       </visual>
       <collision>
+        <origin xyz="0 0 0.125" rpy="0 0 0"/>
         <geometry>
           <mesh filename="package://aurobot_description/meshes/pa10-green/upper_arm/E1.stl"/>
@@ -34,7 +36,7 @@
       <parent link="pa10_green_elbow_flex_link"/>
       <child link="pa10_green_forearm_roll_link"/>
-      <origin xyz="0 0 0.264" rpy="0 0 0"/>
+      <origin xyz="0 0 0.125" rpy="0 0 0"/>
       <axis xyz="0 1 0"/>
-      <limit effort="1000.0" lower="-2.3911010752" upper="2.3911010752" velocity="0.2"/>
+      <limit effort="1000.0" lower="-2.39" upper="2.39" velocity="0.2"/>
       <cfm>0.7</cfm>
       <damping>10.0</damping>
@@ -43,5 +45,5 @@
     <link name="pa10_green_forearm_roll_link">
       <inertial>
-        <origin xyz="0 0 0" rpy="0 0 0"/>
+        <origin xyz="0 -0.046 0" rpy="0 0 0"/>
         <mass value="4.31"/>
         <inertia ixx="0.051762"  ixy="-0.000577"  ixz="0.000005" iyy="0.006329" iyz="0.000005" izz="0.051407"/>
@@ -63,7 +65,6 @@
       <child link="${child}"/>
       <axis xyz="0 0 1"/>
-      <origin xyz="0 0 0.261" rpy="0 0 0"/>
-      <!-- BRAYAN (13/07/2017): gran cambio en lower y upper, casi el doble hemos puesto -->
-      <limit effort="1000.0" lower="-4.4505895926" upper="4.4505895926" velocity="0.628"/>
+      <origin xyz="0 0 0.450" rpy="0 0 0"/>
+      <limit effort="1000.0" lower="-2.0" upper="2.0" velocity="0.628"/>
     </joint>
     <!-- extensions-->

File: aurobot_description/urdf/robot-base/trunk/trunk.urdf.xacro (robot description, xacro)
@@ -38,11 +38,16 @@
       <parent link="trunk_link"/>
       <child link="${head_child}"/>
-      <!-- BRAYAN (16-05-2017): Temporalmente puesto como una cabeza adelantada orientada hacia adelante -->
+      <!-- BRAYAN (16/05/2017): Temporalmente puesto como una cabeza adelantada orientada hacia adelante -->
       <!-- <origin xyz="0.045 -0.025 1.71" rpy="-2.2689280276 0 -1.570796327"/> -->
-      <!-- BRAYAN (14/07/2017): posicion a la izquierda.
+      <!-- BRAYAN (14/07/2017): posicion a la izquierda buena para agarres de frente.
         Tiene en Roll (X) 112.4 negativos.
         Tiene en Pitch (Y) 0.
-        Tiene en Yaw (Z) unos 175.7 grados de desviacion -->
-      <origin xyz="0.775 1.540 1.733" rpy="-1.9634954085 0 3.0665434958"/>
+        Tiene en Yaw (Z) unos 175.7 grados de desviacion
+      <origin xyz="0.775 1.545 1.738" rpy="-1.9634954085 0 3.0665434958"/>
+        Nueva prueba (19/07/2017):
+        Tiene en Roll (X) 112 negativos.
+        Tiene en Yaw (Z) unos 176.2 grados de desviacion
+      -->
+      <origin xyz="0.775 1.542 1.735" rpy="-1.9547687622 0 3.075270142"/>
     </joint>
     <joint name="trunk_right_joint" type="fixed">
