Commit message: Still testing camera positions...

File: aurobot_description/urdf/pa10-green/forearm/forearm.urdf.xacro (robot description, xacro)
@@ -15,9 +15,10 @@
     <link name="pa10_green_wrist_flex_link">
       <inertial>
-        <origin xyz="0 0 0" rpy="0 0 0"/>
+        <origin xyz="0 -0.0432 0.03" rpy="0 0 0"/>
         <mass value="3.45"/>
         <inertia ixx="0.076687"  ixy="0.000005"  ixz="0.000960" iyy="0.077392" iyz="0.000005" izz="0.006233"/>
       </inertial>
       <visual>
+        <origin xyz="0 0 0.03" rpy="0 0 0"/>
         <geometry>
           <mesh filename="package://aurobot_description/meshes/pa10-green/forearm/W1.dae"/>
@@ -26,4 +27,5 @@
       </visual>
       <collision>
+        <origin xyz="0 0 0.03" rpy="0 0 0"/>
         <geometry>
           <mesh filename="package://aurobot_description/meshes/pa10-green/forearm/W1.stl"/>
@@ -34,5 +36,5 @@
       <parent link="pa10_green_wrist_flex_link"/>
       <child link="pa10_green_wrist_roll_link"/>
-      <origin xyz="0 0 0.239" rpy="0 0 0"/>
+      <origin xyz="0 0 0.05" rpy="0 0 0"/>
       <axis xyz="0 1 0"/>
       <limit effort="1000.0" lower="-2.8797932658" upper="2.8797932658" velocity="0.628"/>
@@ -42,9 +44,10 @@
     <link name="pa10_green_wrist_roll_link">
       <inertial>
-        <origin xyz="0 0 0" rpy="0 0 0"/>
+        <origin xyz="0 0.003 -0.0175" rpy="0 0 0"/>
         <mass value="1.46"/>
         <inertia ixx="0.012500"  ixy="0.000005"  ixz="0.000005" iyy="0.011431" iyz="0.000005" izz="0.012500"/>
       </inertial>
       <visual>
+        <origin xyz="0 0.0 -0.0175" rpy="0 0 0"/>
         <geometry>
           <mesh filename="package://aurobot_description/meshes/pa10-green/forearm/W2.dae"/>
@@ -53,4 +56,5 @@
       </visual>
       <collision>
+        <origin xyz="0 0.0 -0.0175" rpy="0 0 0"/>
         <geometry>
           <mesh filename="package://aurobot_description/meshes/pa10-green/forearm/W2.stl"/>

File: aurobot_description/urdf/pa10-green/upper_arm/upper_arm.urdf.xacro (robot description, xacro)
@@ -15,9 +15,10 @@
     <link name="pa10_green_elbow_flex_link">
       <inertial>
-        <origin xyz="0 0 0" rpy="0 0 0"/>
+        <origin xyz="0 0 0.47" rpy="0 0 0"/>
         <mass value="3.51"/>
         <inertia ixx="0.032979"  ixy="0.000005"  ixz="0.000002" iyy="0.017031" iyz="0.000027" izz="0.022417"/>
       </inertial>
       <visual>
+        <origin xyz="0 0 0.125" rpy="0 0 0"/>
         <geometry>
           <mesh filename="package://aurobot_description/meshes/pa10-green/upper_arm/E1.dae"/>
@@ -26,4 +27,5 @@
       </visual>
       <collision>
+        <origin xyz="0 0 0.125" rpy="0 0 0"/>
         <geometry>
           <mesh filename="package://aurobot_description/meshes/pa10-green/upper_arm/E1.stl"/>
@@ -34,5 +36,5 @@
       <parent link="pa10_green_elbow_flex_link"/>
       <child link="pa10_green_forearm_roll_link"/>
-      <origin xyz="0 0 0.264" rpy="0 0 0"/>
+      <origin xyz="0 0 0.125" rpy="0 0 0"/>
       <axis xyz="0 1 0"/>
       <limit effort="1000.0" lower="-2.3911010752" upper="2.3911010752" velocity="0.2"/>
@@ -43,5 +45,5 @@
     <link name="pa10_green_forearm_roll_link">
       <inertial>
-        <origin xyz="0 0 0" rpy="0 0 0"/>
+        <origin xyz="0 -0.046 0" rpy="0 0 0"/>
         <mass value="4.31"/>
         <inertia ixx="0.051762"  ixy="-0.000577"  ixz="0.000005" iyy="0.006329" iyz="0.000005" izz="0.051407"/>
@@ -63,5 +65,5 @@
       <child link="${child}"/>
       <axis xyz="0 0 1"/>
-      <origin xyz="0 0 0.261" rpy="0 0 0"/>
+      <origin xyz="0 0 0.450" rpy="0 0 0"/>
       <!-- BRAYAN (13/07/2017): gran cambio en lower y upper, casi el doble hemos puesto -->
       <limit effort="1000.0" lower="-4.4505895926" upper="4.4505895926" velocity="0.628"/>

File: aurobot_description/urdf/robot-base/trunk/trunk.urdf.xacro (robot description, xacro)
@@ -43,11 +43,11 @@
         Tiene en Roll (X) 112.4 negativos.
         Tiene en Pitch (Y) 0.
-        Tiene en Yaw (Z) unos 175.7 grados de desviacion
+        Tiene en Yaw (Z) unos 175.7 grados de desviacion -->
       <origin xyz="0.775 1.545 1.738" rpy="-1.9634954085 0 3.0665434958"/>
+      <!--
         Nueva prueba (19/07/2017):
         Tiene en Roll (X) 112 negativos.
-        Tiene en Yaw (Z) unos 176.2 grados de desviacion
-      -->
-      <origin xyz="0.775 1.542 1.735" rpy="-1.9547687622 0 3.075270142"/>
+        Tiene en Yaw (Z) unos 176.2 grados de desviacion -->
+      <!-- <origin xyz="0.775 1.537 1.735" rpy="-1.9547687622 0 3.075270142"/> -->
     </joint>
     <joint name="trunk_right_joint" type="fixed">
