Commit message: Fixed trunk decription so the head link is now positioned in the new pose.

File: aurobot_description/urdf/robot-base/trunk/trunk.urdf.xacro (robot description, xacro)
@@ -40,5 +40,6 @@
       <!-- BRAYAN (16-05-2017): Temporalmente puesto como una cabeza adelantada orientada hacia adelante.
       -1.570796327 0 -1.570796327-->
-      <origin xyz="0.150 0 1.47" rpy="-2.042035225 0 -1.570796327"/>
+      <!-- <origin xyz="0.150 0 1.47" rpy="-2.042035225 0 -1.570796327"/> -->
+      <origin xyz="0.045 0 1.71" rpy="-2.042035225 0 -1.570796327"/>
     </joint>
     <joint name="trunk_right_joint" type="fixed">

Commit message: Updated robot head link pose to make it correspond with the actual camera set.

File: aurobot_description/urdf/robot-base/trunk/trunk.urdf.xacro (robot description, xacro)
@@ -41,5 +41,5 @@
       -1.570796327 0 -1.570796327-->
       <!-- <origin xyz="0.150 0 1.47" rpy="-2.042035225 0 -1.570796327"/> -->
-      <origin xyz="0.045 0 1.71" rpy="-2.042035225 0 -1.570796327"/>
+      <origin xyz="0.045 0 1.71" rpy="-2.2689280276 0 -1.570796327"/>
     </joint>
     <joint name="trunk_right_joint" type="fixed">

Commit message: Camera point of view changed to be placed on the left of the robot.

File: aurobot_description/urdf/robot-base/trunk/trunk.urdf.xacro (robot description, xacro)
@@ -40,6 +40,7 @@
       <!-- BRAYAN (16-05-2017): Temporalmente puesto como una cabeza adelantada orientada hacia adelante.
       -1.570796327 0 -1.570796327-->
-      <!-- <origin xyz="0.150 0 1.47" rpy="-2.042035225 0 -1.570796327"/> -->
-      <origin xyz="0.045 0 1.71" rpy="-2.2689280276 0 -1.570796327"/>
+      <!-- <origin xyz="0.045 -0.025 1.71" rpy="-2.2689280276 0 -1.570796327"/> -->
+      <!-- BRAYAN (04/07/2017): posicion a la izquierda -->
+      <origin xyz="0.69 1.366 1.765" rpy="-1.9722220548 0 3.1415926536"/>
     </joint>
     <joint name="trunk_right_joint" type="fixed">

Commit message: Nice camera configuration for grasping the milk box! Added a pre grasping and a post grasping palm position so the whole grasping process is now divided in sub steps.

File: aurobot_description/urdf/robot-base/trunk/trunk.urdf.xacro (robot description, xacro)
@@ -40,7 +40,9 @@
       <!-- BRAYAN (16-05-2017): Temporalmente puesto como una cabeza adelantada orientada hacia adelante -->
       <!-- <origin xyz="0.045 -0.025 1.71" rpy="-2.2689280276 0 -1.570796327"/> -->
-      <!-- BRAYAN (10/07/2017): posicion a la izquierda. Tiene en Roll (X) 109 negativos.
-        Tiene rotado en Yaw (Z) unos 180 + 1 grados de desviacion -->
-      <origin xyz="0.71 1.526 1.793" rpy="-2.0071286398 0 3.1538099584"/>
+      <!-- BRAYAN (14/07/2017): posicion a la izquierda.
+        Tiene en Roll (X) 112.4 negativos.
+        Tiene en Pitch (Y) 0.
+        Tiene en Yaw (Z) unos 175.7 grados de desviacion -->
+      <origin xyz="0.775 1.540 1.733" rpy="-1.9634954085 0 3.0665434958"/>
     </joint>
     <joint name="trunk_right_joint" type="fixed">

Commit message: Last modificacions before summer holidays: - Re position left camera coordinates - Minor changes to the executables

File: aurobot_description/urdf/robot-base/trunk/trunk.urdf.xacro (robot description, xacro)
@@ -44,5 +44,5 @@
         Tiene en Pitch (Y) 0.
         Tiene en Yaw (Z) unos 175.7 grados de desviacion -->
-      <origin xyz="0.775 1.545 1.738" rpy="-1.9634954085 0 3.0665434958"/>
+      <origin xyz="0.778 1.548 1.742" rpy="-1.9634954085 0 3.0665434958"/>
       <!--
         Nueva prueba (19/07/2017):
