Commit message: Changed the MoveIt! planner. Some TODOs added.

File: aurobot_description/urdf/pa10-green/upper_arm/upper_arm.urdf.xacro (robot description, xacro)
@@ -51,6 +51,5 @@
       <visual>
         <geometry>
-          <!-- BRAYAN (22/11/2017): Escalamos esta pieza que en el STL mide 289.6 y en la realidad ronda 293.02 -->
-          <mesh filename="package://aurobot_description/meshes/pa10-green/upper_arm/pa10_04.stl" scale="1 1 1.1"/>
+          <mesh filename="package://aurobot_description/meshes/pa10-green/upper_arm/pa10_04.stl"/>
         </geometry>
         <material name="blue"/>
@@ -58,5 +57,5 @@
       <collision>
         <geometry>
-          <mesh filename="package://aurobot_description/meshes/pa10-green/upper_arm/pa10_04.stl" scale="1 1 1.1"/>
+          <mesh filename="package://aurobot_description/meshes/pa10-green/upper_arm/pa10_04.stl"/>
         </geometry>
       </collision>
